File: hardware/zom/zom1.kicad_pcb (KiCad board)
At the start: 2 copper layers, 2 parts, among them U1 ESP32-WROOM, U2 RFM95HW

Commit message: update
Parts:
- added C1: 10 uF, Capacitors_THT:C_Disc_D3.0mm_W1.6mm_P2.50mm, F.Cu at (86.4, 53.3)
- added C2: 22 uF, Capacitors_THT:C_Disc_D3.0mm_W1.6mm_P2.50mm, F.Cu at (74.9, 53.3)
- added C3: C, Capacitors_THT:C_Disc_D3.0mm_W1.6mm_P2.50mm, F.Cu at (74.9, 116.8)
- added C4: C, Capacitors_THT:C_Disc_D3.0mm_W1.6mm_P2.50mm, F.Cu at (72.4, 38.1)
- added C5: 10 uF, Capacitors_THT:C_Disc_D3.0mm_W1.6mm_P2.50mm, F.Cu at (90.2, 67.3)
- added C6: 22 uF, Capacitors_THT:C_Disc_D3.0mm_W1.6mm_P2.50mm, F.Cu at (95.2, 61.0)
- added J1: Conn_01x03, Socket_Strips:Socket_Strip_Straight_1x03_Pitch2.54mm, F.Cu at (31.8, 111.8)
- added J10: Conn_01x06, Pin_Headers:Pin_Header_Straight_1x06_Pitch2.54mm, F.Cu at (26.7, 82.5)
- added J11: Conn_01x04, TerminalBlocks_Phoenix:TerminalBlock_Phoenix_PT-3.5mm_4pol, F.Cu at (91.4, 100.3)
- added J12: Conn_01x04, Pin_Headers:Pin_Header_Straight_1x04_Pitch2.54mm, F.Cu at (47.0, 108.0)
- added J13: Conn_01x15, Socket_Strips:Socket_Strip_Straight_1x15_Pitch2.54mm, F.Cu at (74.9, 59.7)
- added J14: Conn_01x04, Pin_Headers:Pin_Header_Straight_1x04_Pitch2.54mm, F.Cu at (90.2, 85.1)
- added J15: Conn_01x08, Socket_Strips:Socket_Strip_Straight_1x08_Pitch2.54mm, F.Cu at (67.3, 55.9)
- added J2: Conn_01x07, Pin_Headers:Pin_Header_Straight_1x07_Pitch2.54mm, F.Cu at (82.5, 71.1)
- added J3: Conn_01x02, TerminalBlocks_Phoenix:TerminalBlock_Phoenix_PT-3.5mm_2pol, F.Cu at (95.2, 48.3)
- added J4: Conn_01x07, Pin_Headers:Pin_Header_Straight_1x07_Pitch2.54mm, F.Cu at (57.1, 58.4)
- added J5: Conn_01x04, Pin_Headers:Pin_Header_Straight_1x04_Pitch2.54mm, F.Cu at (41.9, 64.8)
- added J6: Conn_01x03, Pin_Headers:Pin_Header_Straight_1x03_Pitch2.54mm, F.Cu at (82.5, 59.7)
- added J7: Conn_01x01, Pin_Headers:Pin_Header_Straight_1x01_Pitch2.54mm, F.Cu at (45.7, 100.3)
- added J8: Conn_01x04, TerminalBlocks_Phoenix:TerminalBlock_Phoenix_PT-3.5mm_4pol, F.Cu at (41.9, 44.5)
- added J9: Conn_01x03, TerminalBlocks_Phoenix:TerminalBlock_Phoenix_PT-3.5mm_3pol, F.Cu at (33.0, 104.1)
- added Q1: Q_NPN_CBE, TO_SOT_Packages_THT:TO-92_Molded_Narrow, F.Cu at (64.8, 119.4)
- added Q2: Q_NPN_CBE, TO_SOT_Packages_THT:TO-92_Molded_Narrow, F.Cu at (85.1, 110.5)
- added R1: 10K, Resistors_THT:R_Axial_DIN0204_L3.6mm_D1.6mm_P1.90mm_Vertical, F.Cu at (53.3, 120.7)
- added R2: R, Resistors_THT:R_Axial_DIN0204_L3.6mm_D1.6mm_P1.90mm_Vertical, F.Cu at (64.8, 110.5)
- added R3: R, Resistors_THT:R_Axial_DIN0204_L3.6mm_D1.6mm_P1.90mm_Vertical, F.Cu at (92.7, 76.2)
- added R4: 10K, Resistors_THT:R_Axial_DIN0204_L3.6mm_D1.6mm_P1.90mm_Vertical, F.Cu at (64.8, 47.0)
- added R5: R, Resistors_THT:R_Axial_DIN0204_L3.6mm_D1.6mm_P1.90mm_Vertical, F.Cu at (29.2, 68.6)
- added R6: R, Resistors_THT:R_Axial_DIN0204_L3.6mm_D1.6mm_P1.90mm_Vertical, F.Cu at (43.2, 55.9)
- added R7: R, Resistors_THT:R_Axial_DIN0204_L3.6mm_D1.6mm_P1.90mm_Vertical, F.Cu at (53.3, 110.5)
- added SW1: SW_Push, Buttons_Switches_THT:SW_PUSH_6mm, F.Cu at (74.9, 106.7)
- added SW2: SW_Push, Buttons_Switches_THT:SW_PUSH_6mm, F.Cu at (73.7, 43.2)
- moved U2 64.5 mm to (30.5, 82.5)
- moved U1 59.1 mm to (61.0, 90.2)
Connections:
- U1 pad 1: Net-(U1-Pad1) -> GND
- U1 pad 10: Net-(U1-Pad10) -> 25
- U1 pad 11: Net-(U1-Pad11) -> 26
- U1 pad 12: Net-(U1-Pad12) -> 27/SAT_SLEEP
- U1 pad 13: Net-(U1-Pad13) -> 14
- U1 pad 14: Net-(U1-Pad14) -> 12
- U1 pad 15: Net-(U1-Pad15) -> GND
- U1 pad 16: Net-(U1-Pad16) -> 13
- U1 pad 17: Net-(U1-Pad17) -> (no net)
- U1 pad 18: Net-(U1-Pad18) -> (no net)
- U1 pad 19: Net-(U1-Pad19) -> (no net)
- U1 pad 2: Net-(U1-Pad2) -> 22
- U1 pad 20: Net-(U1-Pad20) -> (no net)
- U1 pad 21: Net-(U1-Pad21) -> (no net)
- U1 pad 22: Net-(U1-Pad22) -> (no net)
- U1 pad 23: Net-(U1-Pad23) -> (no net)
- U1 pad 24: Net-(U1-Pad24) -> 2
- U1 pad 25: Net-(U1-Pad25) -> 0
- U1 pad 26: Net-(U1-Pad26) -> SDA
- U1 pad 27: Net-(U1-Pad27) -> SCL
- U1 pad 28: Net-(U1-Pad28) -> 17
- U1 pad 29: Net-(U1-Pad29) -> 5
- U1 pad 3: Net-(U1-Pad3) -> RESET
- U1 pad 30: Net-(U1-Pad30) -> 18
- U1 pad 31: Net-(U1-Pad31) -> 19
- U1 pad 32: Net-(U1-Pad32) -> (no net)
- U1 pad 33: Net-(U1-Pad33) -> 21
- U1 pad 34: Net-(U1-Pad34) -> (no net)
- U1 pad 35: Net-(U1-Pad35) -> (no net)
- U1 pad 36: Net-(U1-Pad36) -> 22
- U1 pad 37: Net-(U1-Pad37) -> 23
- U1 pad 38: Net-(U1-Pad38) -> GND
- U1 pad 39: Net-(U1-Pad39) -> GND
- U1 pad 4: Net-(U1-Pad4) -> (no net)
- U1 pad 5: Net-(U1-Pad5) -> (no net)
- U1 pad 6: Net-(U1-Pad6) -> 34/RX1
- U1 pad 7: Net-(U1-Pad7) -> 35/RX2
- U1 pad 8: Net-(U1-Pad8) -> 32/TX1
- U1 pad 9: Net-(U1-Pad9) -> 33/TX2
- U2 pad 1: Net-(U2-Pad1) -> GND
- U2 pad 10: Net-(U2-Pad10) -> GND
- U2 pad 13: Net-(U2-Pad13) -> 22
- U2 pad 2: Net-(U2-Pad2) -> 19
- U2 pad 3: Net-(U2-Pad3) -> 18
- U2 pad 4: Net-(U2-Pad4) -> 5
- U2 pad 5: Net-(U2-Pad5) -> 12
- U2 pad 6: Net-(U2-Pad6) -> (no net)
- U2 pad 8: Net-(U2-Pad8) -> GND
Other:
- board outline added: 88.9 x 110.5 mm

Commit message: update
Parts:
- added J16: LBO, Pin_Headers:Pin_Header_Straight_1x05_Pitch2.54mm, F.Cu at (49.5, 38.1)
- added J17: VIN2, Pin_Headers:Pin_Header_Straight_1x02_Pitch2.54mm, F.Cu at (33.0, 97.8)
- J1: value Conn_01x03 -> REG:3V3
- J10: value Conn_01x06 -> LBD
- J11: value Conn_01x04 -> UART
- J12: value Conn_01x04 -> dht22
- J13: value Conn_01x15 -> 9602
- J14: value Conn_01x04 -> satx
- J15: value Conn_01x08 -> MISC
- J2: value Conn_01x07 -> prog
- J3: value Conn_01x02 -> VINS
- J4: value Conn_01x07 -> sdcard
- J5: value Conn_01x04 -> oled
- J6: value Conn_01x03 -> REG:5V
- J7: value Conn_01x01 -> ANT
- J8: value Conn_01x04 -> i2c
- J9: value Conn_01x03 -> 1wire
- moved J3 85.9 mm to (24.1, 96.5)
- moved J7 84.7 mm to (64.8, 17.8)
- moved J11 73.3 mm to (26.7, 66.0), turned to 270 degrees
- moved J10 70.8 mm to (64.8, 22.9)
- moved U1 65.4 mm to (34.3, 30.5), turned to 180 degrees
- moved C6 61.1 mm to (34.3, 57.1)
- moved R1 52.6 mm to (45.7, 68.6)
- moved U2 52.2 mm to (47.0, 33.0), turned to 90 degrees
- moved C1 49.5 mm to (40.6, 72.4)
- moved R7 48.7 mm to (40.6, 63.5)
- moved SW1 48.6 mm to (34.3, 80.0)
- moved Q1 47.4 mm to (48.3, 74.9)
- moved J14 46.6 mm to (69.8, 43.2)
- moved Q2 46.2 mm to (48.3, 82.5)
- moved J2 45.5 mm to (45.7, 97.8), turned to 90 degrees
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Connections:
- U1 pad 23: (no net) -> 15
- U2 pad 6: (no net) -> 15
Other:
- board outline removed

Commit message: update
Parts:
- added J18: i2c-b, Pin_Headers:Pin_Header_Straight_1x04_Pitch2.54mm, F.Cu at (165.1, 102.9)
- J5: value oled -> i2c-a
- J8: value i2c -> i2c-c
- moved J8 184.1 mm to (194.3, 125.7), turned to 90 degrees
- moved J11 183.6 mm to (194.3, 141.0), turned to 90 degrees
- moved J9 170.0 mm to (194.3, 110.5), turned to 90 degrees
- moved C6 163.2 mm to (180.3, 130.0), turned to 270 degrees
- moved J15 161.7 mm to (188.6, 121.3), turned to 180 degrees
- moved J2 151.8 mm to (197.5, 95.9), turned to 180 degrees
- moved U1 151.4 mm to (180.3, 70.5)
- moved R7 146.1 mm to (183.5, 94.0), turned to 180 degrees
- moved R5 144.1 mm to (168.3, 109.9), turned to 90 degrees
- moved C1 140.3 mm to (167.6, 132.1), turned to 90 degrees
- moved C5 139.5 mm to (185.4, 132.7), turned to 90 degrees
- moved J3 139.2 mm to (156.8, 138.4)
- moved C2 134.8 mm to (172.2, 129.5), turned to 270 degrees
- moved Q1 132.7 mm to (174.0, 117.5), turned to 180 degrees
- moved R6 132.2 mm to (163.8, 109.9), turned to 90 degrees
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Other:
- board text added: "9602"
- board text added: "oled"

Commit message: update
Parts:
- removed J17: VIN2, Pin_Headers:Pin_Header_Straight_1x02_Pitch2.54mm
- removed J18: i2c-b, Pin_Headers:Pin_Header_Straight_1x04_Pitch2.54mm
- added J19: 9602-b, Pin_Headers:Pin_Header_Straight_1x08_Pitch2.54mm, F.Cu at (75.1, 83.2)
- added R8: R, Resistors_THT:R_Axial_DIN0204_L3.6mm_D1.6mm_P1.90mm_Vertical, F.Cu at (100.3, 89.5)
- J11: value UART -> uart; footprint TerminalBlocks_Phoenix:TerminalBlock_Phoenix_PT-3.5mm_4pol -> TerminalBlocks_Phoenix:TerminalBlock_Phoenix_PT-3.5mm_5pol
- J13: value 9602 -> 9602-a; footprint Socket_Strips:Socket_Strip_Straight_1x15_Pitch2.54mm -> Pin_Headers:Pin_Header_Straight_1x06_Pitch2.54mm
- J15: value MISC -> misc; footprint Socket_Strips:Socket_Strip_Straight_1x08_Pitch2.54mm -> Pin_Headers:Pin_Header_Straight_1x12_Pitch2.54mm
- J16: footprint Pin_Headers:Pin_Header_Straight_1x05_Pitch2.54mm -> Pin_Headers:Pin_Header_Straight_2x03_Pitch2.54mm
- moved J15 110.6 mm to (121.9, 33.0), turned to 0 degrees
- moved R2 97.6 mm to (89.5, 73.7), turned to 270 degrees
- moved C2 95.5 mm to (80.0, 104.8), turned to 0 degrees
- moved J4 93.7 mm to (106.0, 95.2), turned to 270 degrees
- moved R3 91.4 mm to (87.6, 69.8)
- moved C1 91.3 mm to (82.5, 99.1), turned to 270 degrees
- moved Q1 90.3 mm to (96.5, 71.1)
- moved J8 90.1 mm to (119.7, 75.2)
- moved J1 87.5 mm to (92.7, 100.3)
- moved R5 84.9 mm to (97.2, 63.5), turned to 0 degrees
- moved R6 84.9 mm to (92.7, 63.5), turned to 0 degrees
- moved C5 84.6 mm to (110.5, 93.3), turned to 270 degrees
- moved J2 83.2 mm to (114.3, 95.2)
- moved J11 83.0 mm to (119.7, 104.6)
- moved Q2 81.7 mm to (96.5, 76.8), turned to 180 degrees
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Connections:
- net 34/RX1 renamed 34
- net Net-(J10-Pad2) renamed DIO1
- net Net-(J10-Pad5) renamed DIO4
- C1 pad 2: Net-(C1-Pad2) -> GND
- C2 pad 1: Net-(C1-Pad2) -> GND
- C2 pad 2: 22 -> +3V3
- C5 pad 2: Net-(C5-Pad2) -> GND
- C6 pad 1: Net-(C5-Pad2) -> GND
- J1 pad 1: 22 -> +3V3
- J10 pad 1: Net-(J10-Pad1) -> DIO2
- J10 pad 3: Net-(J10-Pad3) -> DIO0
- J10 pad 4: Net-(J10-Pad4) -> +3V3
- J10 pad 6: Net-(J10-Pad6) -> DIO3
- J11 pad 1: 33/TX2 -> +3V3
- J11 pad 2: 35/RX2 -> VIN
- J11 pad 3: 22 -> (no net)
- J11 pad 4: GND -> (no net)
- J12 pad 1: 22 -> +3V3
- J12 pad 2: 25 -> Net-(J12-Pad2)
- J13 pad 3: 32/TX1 -> 13
- J15 pad 2: 22 -> +3V3
- J15 pad 4: 0 -> (no net)
- J15 pad 5: 2 -> (no net)
- J15 pad 6: 13 -> (no net)
- J15 pad 7: 26 -> (no net)
- J15 pad 8: 27/SAT_SLEEP -> (no net)
- J16 pad 1: 12 -> 33
- J16 pad 2: 18 -> 32
- J16 pad 3: 19 -> 26
- J16 pad 4: 5 -> 25
- J16 pad 5: 15 -> DIO5
- J2 pad 4: (no net) -> RXD0
- J2 pad 5: (no net) -> TXD0
- J4 pad 1: 14 -> (no net)
- J4 pad 2: 21 -> (no net)
- J4 pad 4: 22 -> +3V3
- J4 pad 5: 23 -> (no net)
- J4 pad 7: 17 -> (no net)
- J5 pad 1: SDA -> 12/SDA
- J5 pad 2: SCL -> 14/SCL
- J5 pad 3: 22 -> +3V3
- J8 pad 1: SDA -> +3V3
- J8 pad 2: SCL -> GND
- J8 pad 3: 22 -> 12/SDA
- J8 pad 4: GND -> 14/SCL
- J9 pad 1: 22 -> GND
- J9 pad 2: 22 -> Net-(J9-Pad2)
- J9 pad 3: GND -> +3V3
- R1 pad 1: 22 -> +3V3
- R4 pad 1: 22 -> +3V3
- R5 pad 1: 22 -> +3V3
- R5 pad 2: SCL -> 12/SDA
- R6 pad 1: 22 -> +3V3
- R6 pad 2: SDA -> 14/SCL
- R7 pad 1: 22 -> +3V3
- R7 pad 2: 25 -> Net-(J12-Pad2)
- U1 pad 12: 27/SAT_SLEEP -> 27
- U1 pad 13: 14 -> 14/SCL
- U1 pad 14: 12 -> 12/SDA
- U1 pad 2: 22 -> +3V3
- U1 pad 23: 15 -> (no net)
- U1 pad 24: 2 -> (no net)
- U1 pad 26: SDA -> (no net)
- U1 pad 27: SCL -> (no net)
- U1 pad 28: 17 -> (no net)
- U1 pad 29: 5 -> (no net)
- U1 pad 30: 18 -> (no net)
- U1 pad 31: 19 -> (no net)
- U1 pad 33: 21 -> (no net)
- U1 pad 34: (no net) -> RXD0
- U1 pad 35: (no net) -> TXD0
- U1 pad 36: 22 -> (no net)
- U1 pad 37: 23 -> (no net)
- U1 pad 7: 35/RX2 -> (no net)
- U1 pad 8: 32/TX1 -> 32
- U1 pad 9: 33/TX2 -> 33
- U2 pad 11: Net-(J10-Pad4) -> DIO3
- U2 pad 13: 22 -> +3V3
- U2 pad 14: Net-(J10-Pad1) -> DIO0
- U2 pad 16: Net-(J10-Pad3) -> DIO2
- U2 pad 2: 19 -> 32
- U2 pad 3: 18 -> 33
- U2 pad 4: 5 -> 25
- U2 pad 5: 12 -> 26
- U2 pad 6: 15 -> 27
- U2 pad 7: Net-(J10-Pad6) -> DIO5
Routing:
- net GND: track 0.00 -> 214.3 mm, vias 0 -> 3
- net +3V3: track 0.00 -> 149.1 mm, vias 0 -> 3
- net VIN: track 0.00 -> 57.9 mm
- net 13: track 0.00 -> 44.4 mm, vias 0 -> 1
- net 34: track 0.00 -> 39.1 mm, vias 0 -> 1
- net 14/SCL: track 0.00 -> 38.9 mm, vias 0 -> 1
- net DTR: track 0.00 -> 38.2 mm
- net 33: track 0.00 -> 36.9 mm
- net 12/SDA: track 0.00 -> 36.3 mm
- net 32: track 0.00 -> 36.0 mm
- net 26: track 0.00 -> 31.1 mm
- net 25: track 0.00 -> 30.9 mm
- net 0: track 0.00 -> 30.2 mm
- net RTS: track 0.00 -> 29.8 mm, vias 0 -> 1
- net 27: track 0.00 -> 25.5 mm
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Other:
- board outline added: 51.5 x 76.2 mm
- net class power added: clearance 0.2, trace_width 0.35, via_dia 0.6, via_drill 0.4
