File: hardware/zom/zom1.kicad_pcb (KiCad board)
At the start: 2 copper layers, 51.5 x 76.2 mm, 37 parts, among them J1 REG:3V3, J10 LBD, J11 uart, J12 dht22, J13 9602-a, J14 satx, J15 misc, J16 LBO, J19 9602-b, J2 prog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

Commit message: update
Connections:
- U1 pad 33: 23/SAT_SLEEP -> (no net)
- U1 pad 37: (no net) -> 23/SAT_SLEEP
Routing:
- net RX0: track 0.00 -> 49.0 mm, vias 0 -> 5
- net TX0: track 0.00 -> 47.8 mm, vias 0 -> 5
- net RESET: track 22.5 -> 63.1 mm, vias 0 -> 3
- net +3V3: track 169.2 -> 203.7 mm, vias 3 -> 6
- net 14/SCL: track 21.4 -> 49.3 mm, vias 0 -> 2
- net 23/SAT_SLEEP: track 79.4 -> 91.1 mm
- net 12/SDA: track 37.6 -> 40.0 mm
- net 13: track 53.4 -> 55.5 mm
- net GND: track 256.5 -> 255.0 mm
- net 0: track 36.7 -> 37.8 mm

Commit message: update
Parts:
- added D1: D, Diodes_THT:D_DO-201_P5.08mm_Vertical_AnodeUp, F.Cu at (105.4, 85.0)
- added D2: D, Diodes_THT:D_DO-201_P5.08mm_Vertical_AnodeUp, F.Cu at (84.8, 94.2)
Connections:
- C1 pad 1: VIN -> Net-(C1-Pad1)
- J1 pad 3: VIN -> Net-(C1-Pad1)
- J11 pad 3: (no net) -> 21
- J11 pad 4: (no net) -> 19
- J15 pad 1: 35 -> (no net)
- J15 pad 10: (no net) -> +3V3
- J15 pad 11: VIN -> 14/SCL
- J15 pad 12: (no net) -> 12/SDA
- J15 pad 2: +3V3 -> (no net)
- J15 pad 3: GND -> (no net)
- J15 pad 4: 23/SAT_SLEEP -> (no net)
- J15 pad 9: (no net) -> GND
- J2 pad 3: VIN -> VBUS
- J9 pad 2: Net-(J9-Pad2) -> 22
- R8 pad 2: Net-(J9-Pad2) -> 22
- U1 pad 31: (no net) -> 19
- U1 pad 33: (no net) -> 21
- U1 pad 36: (no net) -> 22
- U1 pad 7: 35 -> (no net)
Routing:
- net 21: track 0.00 -> 65.4 mm
- net 19: track 0.00 -> 58.7 mm
- net 22: track 0.00 -> 55.2 mm, vias 0 -> 3
- net Net-(C1-Pad1): track 0.00 -> 47.7 mm, vias 0 -> 1
- net 35: track 28.9 -> 0.00 mm, vias 2 -> 0
- net GND: track 255.0 -> 270.0 mm
- net Net-(J9-Pad2): track 11.2 -> 0.00 mm
- net 14/SCL: track 49.3 -> 56.5 mm
- net VBUS: track 0.00 -> 7.01 mm
- net 23/SAT_SLEEP: track 91.1 -> 84.7 mm, vias 2 -> 4
- net 12/SDA: track 40.0 -> 46.0 mm
- net DTR: track 38.2 -> 34.4 mm, vias 0 -> 2
- net RTS: track 31.9 -> 28.2 mm
- net +3V3: track 203.7 -> 200.2 mm
- net 17: track 76.2 -> 78.4 mm
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
Commit message: update
Connections:
- J15 pad 1: (no net) -> +5V
- J15 pad 2: (no net) -> 35
- J15 pad 3: (no net) -> 21
- J15 pad 4: (no net) -> 19
- J15 pad 5: (no net) -> 5
- J15 pad 6: (no net) -> 2
- J15 pad 7: (no net) -> 0
- J15 pad 8: (no net) -> VIN
- U1 pad 24: (no net) -> 2
- U1 pad 29: (no net) -> 5
- U1 pad 7: (no net) -> 35
Routing:
- net +5V: track 44.1 -> 123.6 mm, vias 1 -> 2
- net VIN: track 57.0 -> 110.4 mm
- net GND: track 270.0 -> 311.6 mm, vias 5 -> 6
- net 35: track 0.00 -> 34.4 mm, vias 0 -> 3
- net 2: track 0.00 -> 22.3 mm, vias 0 -> 4
- net 22: track 55.2 -> 69.9 mm
- net 5: track 0.00 -> 14.0 mm, vias 0 -> 1
- net 0: track 37.8 -> 47.6 mm
- net 21: track 65.4 -> 73.3 mm
- net 19: track 58.7 -> 65.1 mm, vias 0 -> 1
- net 18: track 22.5 -> 26.9 mm
- net 34: track 35.7 -> 37.0 mm
