File: hardware/zom/zom1.kicad_pcb (KiCad board)
At the start: 2 copper layers, 51.6 x 75.9 mm, 39 parts, among them J1 REG:3V3, J10 LBD, J11 uart, J12 dht22, J13 9602-a, J14 satx, J15 misc, J16 LBO, J19 9602-b, J2 prog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

Commit message: update
Connections:
- J5 pad 3: +3V3 -> GND
- J5 pad 4: GND -> +3V3
Routing:
- net 14/SCL: track 56.5 -> 52.3 mm
- net GND: track 311.6 -> 307.9 mm
- net +3V3: track 200.2 -> 198.8 mm, vias 6 -> 7
- net RESET: track 63.1 -> 64.1 mm

Commit message: update
Parts:
- moved J1 5.34 mm to (87.4, 100.1), turned to 90 degrees
- moved J6 0.43 mm to (107.6, 100.0)
Connections:
- J1 pad 1: +3V3 -> Net-(C1-Pad1)
- J1 pad 3: Net-(C1-Pad1) -> +3V3
- J6 pad 1: +5V -> VIN
- J6 pad 3: VIN -> +5V
Routing:
- net +5V: track 123.6 -> 126.4 mm, vias 2 -> 3
- net GND: track 307.9 -> 310.2 mm
- net +3V3: track 198.8 -> 200.7 mm, vias 7 -> 8
- net VIN: track 110.4 -> 112.2 mm

Commit message: update
Other:
- board text added: "ZOM-B-COM"
- board text added: "http://edgecollective.io/zom-b-com"
- board text added: "ver 0.1"
Changed lines of the file:
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@@
     (area 72.924599 30.404999 124.636601 106.501001)
     (thickness 1.6)
-    (drawings 24)
+    (drawings 27)
     (tracks 710)
     (zones 0)
@@
     )
   )
+  (gr_text "ver 0.1" (at 95.8596 39.3954 90) (layer F.SilkS)
+    (effects (font (size 0.8 0.8) (thickness 0.125)))
+  )
+  (gr_text http://edgecollective.io/zom-b-com (at 97.0788 44.0182) (layer B.SilkS)
+    (effects (font (size 1.5 1.5) (thickness 0.25)) (justify mirror))
+  )
+  (gr_text ZOM-B-COM (at 93.7006 48.5394 90) (layer F.SilkS)
+    (effects (font (size 3 1.6) (thickness 0.3)))
+  )
   (gr_line (start 92.5576 100.0252) (end 106.0196 100.0252) (angle 90) (layer Dwgs.User) (width 0.2))
