File: hardware/zom/zom1.sch (KiCad schematic (older format))
At the start: 2 parts

Commit message: update
Parts:
- added C1: 10 uF, symbol C
- added C2: 22 uF, symbol C
- added C? (x2): C, symbol C
- added J? (x2): Conn_01x03, symbol Conn_01x03
- added J? (x2): Conn_01x07, symbol Conn_01x07
- added J? (x3): Conn_01x04, symbol Conn_01x04
- added J?: Conn_01x01, symbol Conn_01x01
- added J?: Conn_01x12, symbol Conn_01x12
- added J?: Conn_01x02, symbol Conn_01x02
- added Q? (x2): Q_NPN_CBE, symbol Q_NPN_CBE
- added R? (x5): R, symbol R
- added R? (x2): 10K, symbol R
- added SW? (x2): SW_Push, symbol SW_Push
- U1: renamed from U?; footprint ESP32-footprints-Lib:ESP32-WROOM -> zom:ESP32-WROOM
- U2: renamed from U?; footprint mysensors_radios:RFM69HW_SMD_ThroughHole_Handsoldering -> zom:RFM95
Connections:
- net GND: now reaches U2.1 (GND)
- net GND: now also U1.1 (GND), U1.15 (GND), U1.38 (GND), U1.39 (GND-PAD), U2.10 (GND), U2.8 (GND), C?.2, C?.2, J?.1 (Pin_1), J?.2 (Pin_2), J?.2 (Pin_2), J?.3 (Pin_3), J?.3 (Pin_3), J?.3 (Pin_3), J?.4 (Pin_4), J?.4 (Pin_4), J?.4 (Pin_4), J?.6 (Pin_6), SW?.1, SW?.1
- net +3V3: now reaches U2.13 (3.3V)
- net +3V3: now also U1.2 (3V3), U1.36 (IO22), C2.2, J?.1 (Pin_1), J?.1 (Pin_1), J?.1 (Pin_1), J?.2 (Pin_2), J?.2 (Pin_2), J?.3 (Pin_3), J?.3 (Pin_3), J?.4 (Pin_4), R?.1, R?.1, R?.1, R?.1, R?.1
- net 19: now reaches U2.2 (MISO)
- net 19: now also U1.31 (IO19)
- net 18: now reaches U2.3 (MOSI)
- net 18: now also U1.30 (IO18)
- net 5: now reaches U2.4 (SCK)
- net 5: now also U1.29 (IO5)
- net 12: now reaches U2.5 (NSS)
- net 12: now also U1.14 (IO12)
- net at U2.9 (ANA): now also J?.1 (Pin_1)
- net 25: now reaches U1.10 (IO25)
- net 26: now reaches U1.11 (IO26)
- net 26: now also J?.7 (Pin_7)
- net 27: now reaches U1.12 (IO27)
- net 27: now also J?.8 (Pin_8)
- net 14: now reaches U1.13 (IO14)
- net 14: now also J?.1 (Pin_1)
- net 13: now reaches U1.16 (IO13)
- net 13: now also J?.6 (Pin_6)
- net 15: now reaches U1.23 (IO15)
- net 2: now reaches U1.24 (IO2)
- net 2: now also J?.5 (Pin_5)
- net 0: now reaches U1.25 (IO0)
- net 0: now also C?.1, J?.4 (Pin_4), Q?.1 (C), R?.2, SW?.2
- net SDA: now reaches U1.26 (IO4)
- net SDA: now also J?.1 (Pin_1), J?.1 (Pin_1), R?.2
- net SCL: now reaches U1.27 (IO16)
- net SCL: now also J?.2 (Pin_2), J?.2 (Pin_2), R?.2
- net 17: now reaches U1.28 (IO17)
- net 17: now also J?.7 (Pin_7)
- net RESET: now reaches U1.3 (EN)
- net RESET: now also C?.1, Q?.1 (C), R?.2, SW?.2
- net 21: now reaches U1.33 (IO21)
- net 21: now also J?.2 (Pin_2)
- net RXD0: now reaches U1.34 (RXD0)
- net TXD0: now reaches U1.35 (TXD0)
- net 23: now reaches U1.37 (IO23)
- net 23: now also J?.5 (Pin_5)
- net 34: now reaches U1.6 (IO34)
- net 34: now also J?.11 (Pin_11)
- net 35: now reaches U1.7 (IO35)
- net 35: now also J?.12 (Pin_12)
- net 32: now reaches U1.8 (IO32)
- net 32: now also J?.9 (Pin_9)
- net 33: now reaches U1.9 (IO33)
- net 33: now also J?.10 (Pin_10), J?.2 (Pin_2), R?.2
- new net: C1.2, C2.1
- new net: Q?.2 (B), R?.1 (x2)
- new net DTR: J?.7 (Pin_7), Q?.3 (E), R?.2
- new net RTS: J?.6 (Pin_6), Q?.3 (E), R?.2
- new net RX0: J?.4 (Pin_4)
- new net TX0: J?.5 (Pin_5)
- new net VIN: C1.1, J?.1 (Pin_1), J?.1 (Pin_1), J?.3 (Pin_3), J?.3 (Pin_3)
Other:
- note added: "1-wire"
- note added: "Auto-reset\n(if using CP2104)"
- note added: "OLED DISPLAY"
- note added: "Power In"
- note added: "Programming"
- note added: "Regulator: VX7803"
- note added: "SD Card"
- note added: "i2c"
- note added: "i2c pullups"
- moved on the sheet: U1, U2

Commit message: update
Parts:
- removed J?: Conn_01x12, symbol Conn_01x12
- added C?: 10 uF, symbol C
- added C?: 22 uF, symbol C
- added J?: Conn_01x03, symbol Conn_01x03
- added J?: Conn_01x15, symbol Conn_01x15
- added J? (x2): Conn_01x04, symbol Conn_01x04
- added J?: Conn_01x05, symbol Conn_01x05
Connections:
- net +3V3: now also J?.2 (Pin_2), J?.3 (Pin_3), J?.3 (Pin_3)
- net 0: now also J?.4 (Pin_4)
- net 2: now also J?.5 (Pin_5)
- net 25: now also J?.2 (Pin_2), R?.2
- net GND: now also J?.15 (Pin_15), J?.2 (Pin_2), J?.3 (Pin_3), J?.4 (Pin_4), J?.4 (Pin_4), J?.6 (Pin_6), J?.8 (Pin_8)
- net VIN: now also C?.1, J?.1 (Pin_1), J?.3 (Pin_3)
- net 13 renamed 13/SAT_SLEEP
- net 13/SAT_SLEEP: now also J?.13 (Pin_13)
- net 26 renamed 26/RX3
- net 26/RX3: now also J?.1 (Pin_1)
- net 27 renamed 27/TX3
- net 27/TX3: now also J?.2 (Pin_2)
- net 32 renamed 32/TX1
- net 32/TX1: now also J?.2 (Pin_2)
- removed net 33: J?.2 (Pin_2), R?.2, U1.9 (IO33)
- net 34 renamed 34/RX1
- net 34/RX1: now also J?.3 (Pin_3)
- net 35 renamed 35/RX2
- net 35/RX2: now also J?.2 (Pin_2)
- new net: C?.1, C?.2
- new net +5V: C?.2, J?.1 (Pin_1), J?.4 (Pin_4), J?.9 (Pin_9)
- new net 33/TX2: J?.1 (Pin_1), U1.9 (IO33)
- new net SAT_5V_OUT: J?.10 (Pin_10)
- new net SAT_CTS: J?.5 (Pin_5)
- new net SAT_LION: J?.14 (Pin_14)
- new net SAT_NETWORK_AVAIL: J?.12 (Pin_12)
- new net SAT_RING_INDICATOR: J?.11 (Pin_11)
- new net SAT_RTS: J?.1 (Pin_1)
Other:
- note added: "DHT22"
- note added: "Iridium 9602"
- note added: "Regulator: VX7803 (3.3V)"
- note added: "Regulator: VX7803 (5V)"
- note removed: "Regulator: VX7803"
- moved on the sheet: J?, U2

Commit message: update
Parts:
- removed J?: Conn_01x04, symbol Conn_01x04
- removed J?: Conn_01x05, symbol Conn_01x05
- added J10: Conn_01x06, Pin_Headers:Pin_Header_Straight_1x06_Pitch2.54mm, symbol Conn_01x06
- added J14: Conn_01x04, Pin_Headers:Pin_Header_Straight_1x04_Pitch2.54mm, symbol Conn_01x04
- added J15: Conn_01x08, Socket_Strips:Socket_Strip_Straight_1x08_Pitch2.54mm, symbol Conn_01x08
- C1, C2: footprint (none) -> Capacitors_THT:C_Disc_D3.0mm_W1.6mm_P2.50mm
- C3, C4, C5, C6: renamed from C?; footprint (none) -> Capacitors_THT:C_Disc_D3.0mm_W1.6mm_P2.50mm
- J1: renamed from J?; footprint (none) -> Socket_Strips:Socket_Strip_Straight_1x03_Pitch2.54mm
- J11, J8: renamed from J?; footprint (none) -> TerminalBlocks_Phoenix:TerminalBlock_Phoenix_PT-3.5mm_4pol
- J12, J5: renamed from J?; footprint (none) -> Pin_Headers:Pin_Header_Straight_1x04_Pitch2.54mm
- J13: renamed from J?; footprint (none) -> Socket_Strips:Socket_Strip_Straight_1x15_Pitch2.54mm
- J2, J4: renamed from J?; footprint (none) -> Pin_Headers:Pin_Header_Straight_1x07_Pitch2.54mm
- J3: renamed from J?; footprint (none) -> TerminalBlocks_Phoenix:TerminalBlock_Phoenix_PT-3.5mm_2pol
- J6: renamed from J?; footprint (none) -> Pin_Headers:Pin_Header_Straight_1x03_Pitch2.54mm
- J7: renamed from J?; footprint (none) -> Pin_Headers:Pin_Header_Straight_1x01_Pitch2.54mm
- J9: renamed from J?; footprint (none) -> TerminalBlocks_Phoenix:TerminalBlock_Phoenix_PT-3.5mm_3pol
- Q1, Q2: renamed from Q?; footprint (none) -> TO_SOT_Packages_THT:TO-92_Molded_Narrow
- R1, R2, R3, R4, R5, R6, R7: renamed from R?; footprint (none) -> Resistors_THT:R_Axial_DIN0204_L3.6mm_D1.6mm_P1.90mm_Vertical
- SW1, SW2: renamed from SW?; footprint (none) -> Buttons_Switches_THT:SW_PUSH_6mm
Connections:
- net +3V3: now also J15.2 (Pin_2)
- net 0: now also J15.4 (Pin_4)
- net 2: now also J15.5 (Pin_5)
- net 32/TX1: now also J13.3 (Pin_3); no longer J13.2 (Pin_2)
- net 34/RX1: now also J13.2 (Pin_2); no longer J13.3 (Pin_3)
- net GND: now also J15.3 (Pin_3)
- net SAT_LION: now also J14.4 (Pin_4)
- net SAT_NETWORK_AVAIL: now also J14.2 (Pin_2)
- net SAT_RING_INDICATOR: now also J14.1 (Pin_1)
- net VIN: now also J15.1 (Pin_1)
- net at U2.11 (DIO3): now also J10.4 (Pin_4)
- net at U2.12 (DIO4): now also J10.5 (Pin_5)
- net at U2.14 (DIO0): now also J10.1 (Pin_1)
- net at U2.15 (DIO1): now also J10.2 (Pin_2)
- net at U2.16 (DIO2): now also J10.3 (Pin_3)
- net at U2.7 (DIO5): now also J10.6 (Pin_6)
- net 13/SAT_SLEEP renamed 13
- net 13: now also J15.6 (Pin_6); no longer J13.13 (Pin_13)
- net 26/RX3 renamed 26
- net 26: now also J15.7 (Pin_7)
- net 27/TX3 renamed 27/SAT_SLEEP
- net 27/SAT_SLEEP: now also J13.13 (Pin_13), J14.3 (Pin_3), J15.8 (Pin_8)
- net SAT_5V_OUT: no longer names the net of J13.10 (Pin_10)
- net SAT_RTS: no longer names the net of J13.1 (Pin_1)
Other:
- note added: "RFM95"
- note added: "UART"
- moved on the sheet: C5, C6, J13, J6

Commit message: update
Parts:
- added J16: LBO, Pin_Headers:Pin_Header_Straight_1x05_Pitch2.54mm, symbol Conn_01x05
- added J17: VIN2, Pin_Headers:Pin_Header_Straight_1x02_Pitch2.54mm, symbol Conn_01x02
- J1: value Conn_01x03 -> REG:3V3
- J10: value Conn_01x06 -> LBD
- J11: value Conn_01x04 -> UART
- J12: value Conn_01x04 -> dht22
- J13: value Conn_01x15 -> 9602
- J14: value Conn_01x04 -> satx
- J15: value Conn_01x08 -> MISC
- J2: value Conn_01x07 -> prog
- J3: value Conn_01x02 -> VINS
- J4: value Conn_01x07 -> sdcard
- J5: value Conn_01x04 -> oled
- J6: value Conn_01x03 -> REG:5V
- J7: value Conn_01x01 -> ANT
- J8: value Conn_01x04 -> i2c
- J9: value Conn_01x03 -> 1wire
Connections:
- net 12: now also J16.1 (Pin_1)
- net 15: now also U2.6 (RESET), J16.5 (Pin_5)
- net 18: now also J16.2 (Pin_2)
- net 19: now also J16.3 (Pin_3)
- net 5: now also J16.4 (Pin_4)
- net GND: now also J17.2 (Pin_2)
- net VIN: now also J17.1 (Pin_1)
Other:
- note added: "LORA PINS"
Changed lines of the file:
@@
 P 1000 1350
 F 0 "J1" H 1000 1550 50  0000 C CNN
-F 1 "Conn_01x03" H 1000 1150 50  0000 C CNN
+F 1 "REG:3V3" H 1000 1150 50  0000 C CNN
 F 2 "Socket_Strips:Socket_Strip_Straight_1x03_Pitch2.54mm" H 1000 1350 50  0001 C CNN
 F 3 "" H 1000 1350 50  0001 C CNN
@@
 	1    0    0    -1
 $EndComp
-Text GLabel 6250 3550 0    60   Input ~ 0
+Text GLabel 6250 3600 0    60   Input ~ 0
 15
 $Comp
@@
 P 1550 4950
 F 0 "J2" H 1550 5350 50  0000 C CNN
-F 1 "Conn_01x07" H 1550 4550 50  0000 C CNN
+F 1 "prog" H 1550 4550 50  0000 C CNN
 F 2 "Pin_Headers:Pin_Header_Straight_1x07_Pitch2.54mm" H 1550 4950 50  0001 C CNN
 F 3 "" H 1550 4950 50  0001 C CNN
@@
 P 3750 5550
 F 0 "J4" H 3750 5950 50  0000 C CNN
-F 1 "Conn_01x07" H 3750 5150 50  0000 C CNN
+F 1 "sdcard" H 3750 5150 50  0000 C CNN
 F 2 "Pin_Headers:Pin_Header_Straight_1x07_Pitch2.54mm" H 3750 5550 50  0001 C CNN
 F 3 "" H 3750 5550 50  0001 C CNN
@@
 P 5100 5550
 F 0 "J5" H 5100 5750 50  0000 C CNN
-F 1 "Conn_01x04" H 5100 5250 50  0000 C CNN
+F 1 "oled" H 5100 5250 50  0000 C CNN
 F 2 "Pin_Headers:Pin_Header_Straight_1x04_Pitch2.54mm" H 5100 5550 50  0001 C CNN
 F 3 "" H 5100 5550 50  0001 C CNN
@@
 P 6250 2700
 F 0 "J7" H 6250 2800 50  0000 C CNN
-F 1 "Conn_01x01" H 6250 2600 50  0000 C CNN
+F 1 "ANT" H 6250 2600 50  0000 C CNN
 F 2 "Pin_Headers:Pin_Header_Straight_1x01_Pitch2.54mm" H 6250 2700 50  0001 C CNN
 F 3 "" H 6250 2700 50  0001 C CNN
@@
 P 6850 5850
 F 0 "J8" H 6850 6050 50  0000 C CNN
-F 1 "Conn_01x04" H 6850 5550 50  0000 C CNN
+F 1 "i2c" H 6850 5550 50  0000 C CNN
 F 2 "TerminalBlocks_Phoenix:TerminalBlock_Phoenix_PT-3.5mm_4pol" H 6850 5850 50  0001 C CNN
 F 3 "" H 6850 5850 50  0001 C CNN
@@
 P 6950 4800
 F 0 "J9" H 6950 5000 50  0000 C CNN
-F 1 "Conn_01x03" H 6950 4600 50  0000 C CNN
+F 1 "1wire" H 6950 4600 50  0000 C CNN
 F 2 "TerminalBlocks_Phoenix:TerminalBlock_Phoenix_PT-3.5mm_3pol" H 6950 4800 50  0001 C CNN
 F 3 "" H 6950 4800 50  0001 C CNN
@@
 P 8600 4850
 F 0 "J12" H 8600 5050 50  0000 C CNN
-F 1 "Conn_01x04" H 8600 4550 50  0000 C CNN
+F 1 "dht22" H 8600 4550 50  0000 C CNN
 F 2 "Pin_Headers:Pin_Header_Straight_1x04_Pitch2.54mm" H 8600 4850 50  0001 C CNN
 F 3 "" H 8600 4850 50  0001 C CNN
@@
 P 3200 1100
 F 0 "J3" H 3200 1200 50  0000 C CNN
-F 1 "Conn_01x02" H 3200 900 50  0000 C CNN
+F 1 "VINS" H 3200 900 50  0000 C CNN
 F 2 "TerminalBlocks_Phoenix:TerminalBlock_Phoenix_PT-3.5mm_2pol" H 3200 1100 50  0001 C CNN
 F 3 "" H 3200 1100 50  0001 C CNN
@@
 P 6100 1450
 F 0 "J6" H 6100 1650 50  0000 C CNN
-F 1 "Conn_01x03" H 6100 1250 50  0000 C CNN
+F 1 "REG:5V" H 6100 1250 50  0000 C CNN
 F 2 "Pin_Headers:Pin_Header_Straight_1x03_Pitch2.54mm" H 6100 1450 50  0001 C CNN
 F 3 "" H 6100 1450 50  0001 C CNN
@@
 P 9400 2100
 F 0 "J13" H 9400 2900 50  0000 C CNN
-F 1 "Conn_01x15" H 9400 1300 50  0000 C CNN
+F 1 "9602" H 9400 1300 50  0000 C CNN
 F 2 "Socket_Strips:Socket_Strip_Straight_1x15_Pitch2.54mm" H 9400 2100 50  0001 C CNN
 F 3 "" H 9400 2100 50  0001 C CNN
@@
 P 8250 5800
 F 0 "J11" H 8250 6000 50  0000 C CNN
-F 1 "Conn_01x04" H 8250 5500 50  0000 C CNN
+F 1 "UART" H 8250 5500 50  0000 C CNN
 F 2 "TerminalBlocks_Phoenix:TerminalBlock_Phoenix_PT-3.5mm_4pol" H 8250 5800 50  0001 C CNN
 F 3 "" H 8250 5800 50  0001 C CNN
@@
 	10000 3600 10400 3600
 Wire Wire Line
-	3000 1200 2900 1200
+	2900 1200 3550 1200
 Wire Wire Line
 	6300 1450 6900 1450
@@
 P 9850 2500
 F 0 "J14" H 9850 2700 50  0000 C CNN
-F 1 "Conn_01x04" H 9850 2200 50  0000 C CNN
+F 1 "satx" H 9850 2200 50  0000 C CNN
 F 2 "Pin_Headers:Pin_Header_Straight_1x04_Pitch2.54mm" H 9850 2500 50  0001 C CNN
 F 3 "" H 9850 2500 50  0001 C CNN
@@
 P 7550 3250
 F 0 "J10" H 7550 3550 50  0000 C CNN
-F 1 "Conn_01x06" H 7550 2850 50  0000 C CNN
+F 1 "LBD" H 7550 2850 50  0000 C CNN
 F 2 "Pin_Headers:Pin_Header_Straight_1x06_Pitch2.54mm" H 7550 3250 50  0001 C CNN
 F 3 "" H 7550 3250 50  0001 C CNN
@@
 P 10600 3800
 F 0 "J15" H 10600 4200 50  0000 C CNN
-F 1 "Conn_01x08" H 10600 3300 50  0000 C CNN
+F 1 "MISC" H 10600 3300 50  0000 C CNN
 F 2 "Socket_Strips:Socket_Strip_Straight_1x08_Pitch2.54mm" H 10600 3800 50  0001 C CNN
 F 3 "" H 10600 3800 50  0001 C CNN
@@
 Text Notes 6700 2350 0    60   ~ 0
 RFM95
+$Comp
+L Conn_01x05 J16
+U 1 1 5B8C972B
+P 10150 5250
+F 0 "J16" H 10150 5550 50  0000 C CNN
+F 1 "LBO" H 10150 4950 50  0000 C CNN
+F 2 "Pin_Headers:Pin_Header_Straight_1x05_Pitch2.54mm" H 10150 5250 50  0001 C CNN
+F 3 "" H 10150 5250 50  0001 C CNN
+	1    10150 5250
+	1    0    0    -1
+$EndComp
+Text GLabel 9950 5050 0    60   Input ~ 0
+12
+Text GLabel 9950 5150 0    60   Input ~ 0
+18
+Text GLabel 9950 5250 0    60   Input ~ 0
+19
+Text GLabel 9950 5350 0    60   Input ~ 0
+5
+Text GLabel 9950 5450 0    60   Input ~ 0
+15
+Text Notes 8100 4450 0    60   ~ 0
+DHT22
+Text Notes 9750 4850 0    60   ~ 0
+LORA PINS
+$Comp
+L Conn_01x02 J17
+U 1 1 5B8F1E8D
+P 3750 1100
+F 0 "J17" H 3750 1200 50  0000 C CNN
+F 1 "VIN2" H 3750 900 50  0000 C CNN
+F 2 "Pin_Headers:Pin_Header_Straight_1x02_Pitch2.54mm" H 3750 1100 50  0001 C CNN
+F 3 "" H 3750 1100 50  0001 C CNN
+	1    3750 1100
+	1    0    0    -1
+$EndComp
+Wire Wire Line
+	3000 1100 3550 1100
+Connection ~ 3000 1200
+Connection ~ 3000 1100
+Connection ~ 3700 1000
+Connection ~ 8650 1900
 $EndSCHEMATC

Commit message: update
Parts:
- added J18: i2c-b, Pin_Headers:Pin_Header_Straight_1x04_Pitch2.54mm, symbol Conn_01x04
- J5: value oled -> i2c-a
- J8: value i2c -> i2c-c
Connections:
- net +3V3: now also J18.3 (Pin_3)
- net GND: now also J18.4 (Pin_4)
- net SCL: now also J18.2 (Pin_2)
- net SDA: now also J18.1 (Pin_1)
Other:
- note added: "i2c-a"
- note added: "i2c-b"
- note added: "i2c-c"
- note removed: "OLED DISPLAY"
- note removed: "i2c"
Changed lines of the file:
@@
 P 5100 5550
 F 0 "J5" H 5100 5750 50  0000 C CNN
-F 1 "oled" H 5100 5250 50  0000 C CNN
+F 1 "i2c-a" H 5100 5250 50  0000 C CNN
 F 2 "Pin_Headers:Pin_Header_Straight_1x04_Pitch2.54mm" H 5100 5550 50  0001 C CNN
 F 3 "" H 5100 5550 50  0001 C CNN
@@
 SDA
 Text Notes 4700 5250 0    60   ~ 0
-OLED DISPLAY
+i2c-a
 $Comp
 L +3V3 #PWR017
@@
 P 6850 5850
 F 0 "J8" H 6850 6050 50  0000 C CNN
-F 1 "i2c" H 6850 5550 50  0000 C CNN
+F 1 "i2c-c" H 6850 5550 50  0000 C CNN
 F 2 "TerminalBlocks_Phoenix:TerminalBlock_Phoenix_PT-3.5mm_4pol" H 6850 5850 50  0001 C CNN
 F 3 "" H 6850 5850 50  0001 C CNN
@@
 SDA
 Text Notes 6450 5550 0    60   ~ 0
-i2c
+i2c-c
 $Comp
 L GND #PWR020
@@
 Connection ~ 3700 1000
 Connection ~ 8650 1900
+$Comp
+L Conn_01x04 J18
+U 1 1 5B8F474A
+P 5600 6700
+F 0 "J18" H 5600 6900 50  0000 C CNN
+F 1 "i2c-b" H 5600 6400 50  0000 C CNN
+F 2 "Pin_Headers:Pin_Header_Straight_1x04_Pitch2.54mm" H 5600 6700 50  0001 C CNN
+F 3 "" H 5600 6700 50  0001 C CNN
+	1    5600 6700
+	1    0    0    -1
+$EndComp
+$Comp
+L GND #PWR037
+U 1 1 5B8F4750
+P 5200 6900
+F 0 "#PWR037" H 5200 6650 50  0001 C CNN
+F 1 "GND" H 5200 6750 50  0000 C CNN
+F 2 "" H 5200 6900 50  0001 C CNN
+F 3 "" H 5200 6900 50  0001 C CNN
+	1    5200 6900
+	1    0    0    -1
+$EndComp
+$Comp
+L +3V3 #PWR038
+U 1 1 5B8F4756
+P 4950 6800
+F 0 "#PWR038" H 4950 6650 50  0001 C CNN
+F 1 "+3V3" H 4950 6940 50  0000 C CNN
+F 2 "" H 4950 6800 50  0001 C CNN
+F 3 "" H 4950 6800 50  0001 C CNN
+	1    4950 6800
+	1    0    0    -1
+$EndComp
+Text GLabel 5400 6700 0    60   Input ~ 0
+SCL
+Text GLabel 5400 6600 0    60   Input ~ 0
+SDA
+Text Notes 5200 6400 0    60   ~ 0
+i2c-b
+Wire Wire Line
+	5200 6900 5400 6900
+Wire Wire Line
+	4950 6800 5400 6800
 $EndSCHEMATC

Commit message: update
Parts:
- removed J11: UART, TerminalBlocks_Phoenix:TerminalBlock_Phoenix_PT-3.5mm_4pol, symbol Conn_01x04
- removed J13: 9602, Socket_Strips:Socket_Strip_Straight_1x15_Pitch2.54mm, symbol Conn_01x15
- removed J15: MISC, Socket_Strips:Socket_Strip_Straight_1x08_Pitch2.54mm, symbol Conn_01x08
- removed J16: LBO, Pin_Headers:Pin_Header_Straight_1x05_Pitch2.54mm, symbol Conn_01x05
- removed J17: VIN2, Pin_Headers:Pin_Header_Straight_1x02_Pitch2.54mm, symbol Conn_01x02
- removed J18: i2c-b, Pin_Headers:Pin_Header_Straight_1x04_Pitch2.54mm, symbol Conn_01x04
- added J11: uart, TerminalBlocks_Phoenix:TerminalBlock_Phoenix_PT-3.5mm_5pol, symbol Conn_01x05
- added J13: 9602-a, Pin_Headers:Pin_Header_Straight_1x06_Pitch2.54mm, symbol Conn_01x06
- added J15: misc, Pin_Headers:Pin_Header_Straight_1x12_Pitch2.54mm, symbol Conn_01x12
- added J16: LBO, Pin_Headers:Pin_Header_Straight_2x03_Pitch2.54mm, symbol Conn_02x03_Odd_Even
- added J19: 9602-b, Pin_Headers:Pin_Header_Straight_1x08_Pitch2.54mm, symbol Conn_01x08
- added R8: R, Resistors_THT:R_Axial_DIN0204_L3.6mm_D1.6mm_P1.90mm_Vertical, symbol R
Connections:
- net labels added: 12/SDA, 14/SCL, 16, 27, 32, 33, 34, 35, 4, DIO0, DIO1, DIO2, DIO3, DIO4, DIO5
- net labels removed: 12, 14, 32/TX1, 33/TX2, 34/RX1, 35/RX2, RX0, SCL, SDA, TX0
- wire segments 73 -> 71
Other:
- note added: "RMF95 BREAKOUTS"
- note added: "i2c-screwterm"
- note removed: "LORA PINS"
- note removed: "i2c-b"
- note removed: "i2c-c"
- moved on the sheet: J12, J7, J8, J9, R7, U2
