File: hardware/zom/zom1.sch (KiCad schematic (older format))
At the start: 37 parts, among them J1 REG:3V3, J10 LBD, J11 uart, J12 dht22, J13 9602-a, J14 satx, J15 misc, J16 LBO, J19 9602-b, J2 prog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

Commit message: update
Connections:
- net 23 is gone; now on net 23/SAT_SLEEP: U1.37 (IO23)
- net 23/SAT_SLEEP: no longer U1.33 (IO21)
- new net 21: U1.33 (IO21)
Changed lines of the file:
@@
 Text GLabel 5300 3400 2    60   Input ~ 0
 0
-Text GLabel 5300 2600 2    60   Input ~ 0
+Text GLabel 5300 2200 2    60   Input ~ 0
 23/SAT_SLEEP
 Text GLabel 5300 2500 2    60   Input ~ 0
@@
 Text GLabel 5300 2300 2    60   Input ~ 0
 22
-Text GLabel 5300 2200 2    60   Input ~ 0
-23
+Text GLabel 5300 2600 2    60   Input ~ 0
+21
 Text GLabel 3450 3550 0    60   Input ~ 0
 12/SDA

Commit message: update
Parts:
- added D1, D2: D, Diodes_THT:D_DO-201_P5.08mm_Vertical_AnodeUp, symbol D
Connections:
- net +3V3: now also J15.10 (Pin_10); no longer J15.2 (Pin_2)
- net 12/SDA: now also J15.12 (Pin_12)
- net 14/SCL: now also J15.11 (Pin_11)
- net 19: now also J11.4 (Pin_4)
- net 21: now also J11.3 (Pin_3)
- net 22: now also J9.2 (Pin_2), R8.2
- net 23/SAT_SLEEP: no longer J15.4 (Pin_4)
- net 35: no longer J15.1 (Pin_1)
- net GND: now also J15.9 (Pin_9); no longer J15.3 (Pin_3)
- net VIN: now also D2.2 (A); no longer C1.1, J1.3 (Pin_3), J15.11 (Pin_11), J2.3 (Pin_3)
- new net: C1.1, D1.1 (K), D2.1 (K), J1.3 (Pin_3)
- new net VBUS: D1.2 (A), J2.3 (Pin_3)
Changed lines of the file:
@@
 Text Notes 950  900  0    60   ~ 0
 Regulator: VX7803 (3.3V)
-Text GLabel 2050 1050 2    60   Input ~ 0
+Text GLabel 2150 1050 2    60   Input ~ 0
 VIN
 $Comp
@@
 RTS
 Text GLabel 1350 4850 0    60   Input ~ 0
-VIN
+VBUS
 Text GLabel 1350 5250 0    60   Input ~ 0
 DTR
@@
 L +3V3 #PWR025
 U 1 1 5B891AE7
-P 10500 1450
-F 0 "#PWR025" H 10500 1300 50  0001 C CNN
-F 1 "+3V3" H 10500 1590 50  0000 C CNN
-F 2 "" H 10500 1450 50  0001 C CNN
-F 3 "" H 10500 1450 50  0001 C CNN
-	1    10500 1450
+P 10500 2250
+F 0 "#PWR025" H 10500 2100 50  0001 C CNN
+F 1 "+3V3" H 10500 2390 50  0000 C CNN
+F 2 "" H 10500 2250 50  0001 C CNN
+F 3 "" H 10500 2250 50  0001 C CNN
+	1    10500 2250
 	1    0    0    -1
 $EndComp
@@
 	1    0    0    -1
 $EndComp
-Text GLabel 10900 1650 0    60   Input ~ 0
-23/SAT_SLEEP
 Text Notes 7200 5450 0    60   ~ 0
 DHT22
@@
 Text GLabel 3550 5250 0    60   Input ~ 0
 15
-Text GLabel 10900 1350 0    60   Input ~ 0
-35
-Text GLabel 10900 2350 0    60   Input ~ 0
-VIN
 Text GLabel 6900 6050 0    60   Input ~ 0
 18
@@
 L GND #PWR037
 U 1 1 5B891B40
-P 10600 1550
-F 0 "#PWR037" H 10600 1300 50  0001 C CNN
-F 1 "GND" H 10600 1400 50  0000 C CNN
-F 2 "" H 10600 1550 50  0001 C CNN
-F 3 "" H 10600 1550 50  0001 C CNN
-	1    10600 1550
+P 10200 2150
+F 0 "#PWR037" H 10200 1900 50  0001 C CNN
+F 1 "GND" H 10200 2000 50  0000 C CNN
+F 2 "" H 10200 2150 50  0001 C CNN
+F 3 "" H 10200 2150 50  0001 C CNN
+	1    10200 2150
 	1    0    0    -1
 $EndComp
@@
 	9200 2400 9650 2400
 Wire Wire Line
-	6050 7000 6550 7000
-Wire Wire Line
 	8400 1700 9200 1700
 Wire Wire Line
@@
 Wire Wire Line
 	6300 1450 6900 1450
-Wire Wire Line
-	10500 1450 10900 1450
 Connection ~ 7100 6050
 Wire Wire Line
-	7250 6050 6900 6050
-Wire Wire Line
-	7250 5850 7250 6050
-Wire Wire Line
-	7500 5850 7250 5850
+	6900 6050 7250 6050
+Wire Wire Line
+	7250 6050 7250 5850
+Wire Wire Line
+	7250 5850 7500 5850
 Wire Wire Line
 	7100 5750 7500 5750
@@
 	1200 1450 1200 1650
 Wire Wire Line
-	1200 1050 2050 1050
+	1200 1050 1850 1050
 Wire Wire Line
 	1200 1250 1200 1050
@@
 Connection ~ 1400 1350
 Connection ~ 2950 -750
-Wire Wire Line
-	10900 1550 10600 1550
+Text GLabel 6450 5600 2    60   Input ~ 0
+22
+Text GLabel 2150 700  2    60   Input ~ 0
+VBUS
+Wire Wire Line
+	1850 1050 1850 700
+$Comp
+L D D1
+U 1 1 5B91BD42
+P 2000 700
+F 0 "D1" H 2000 800 50  0000 C CNN
+F 1 "D" H 2000 600 50  0000 C CNN
+F 2 "Diodes_THT:D_DO-201_P5.08mm_Vertical_AnodeUp" H 2000 700 50  0001 C CNN
+F 3 "" H 2000 700 50  0001 C CNN
+	1    2000 700
+	1    0    0    -1
+$EndComp
+$Comp
+L D D2
+U 1 1 5B91BFA9
+P 2000 1050
+F 0 "D2" H 2000 1150 50  0000 C CNN
+F 1 "D" H 2000 950 50  0000 C CNN
+F 2 "Diodes_THT:D_DO-201_P5.08mm_Vertical_AnodeUp" H 2000 1050 50  0001 C CNN
+F 3 "" H 2000 1050 50  0001 C CNN
+	1    2000 1050
+	1    0    0    -1
+$EndComp
+Connection ~ 1850 1050
+Connection ~ 1850 700
+Text GLabel 6550 7000 0    60   Input ~ 0
+21
+Text GLabel 6550 7100 0    60   Input ~ 0
+19
+Text GLabel 10900 2350 0    60   Input ~ 0
+14/SCL
+Text GLabel 10900 2450 0    60   Input ~ 0
+12/SDA
+Wire Wire Line
+	10900 2250 10500 2250
+Wire Wire Line
+	10900 2150 10200 2150
 $EndSCHEMATC

Commit message: update
Connections:
- net +5V: now also J15.1 (Pin_1)
- net 0: now also J15.7 (Pin_7)
- net 19: now also J15.4 (Pin_4)
- net 2: now also J15.6 (Pin_6)
- net 21: now also J15.3 (Pin_3)
- net 35: now also J15.2 (Pin_2)
- net 5: now also J15.5 (Pin_5)
- net VIN: now also J15.8 (Pin_8)
Other:
- moved on the sheet: J10, J15, J16, J7, U2
Changed lines of the file:
@@
 L RFM95HW U2
 U 1 1 5B886D30
-P 6950 3900
-F 0 "U2" H 6600 4150 40  0000 C CNN
-F 1 "RFM95HW" H 7200 3150 40  0000 C CNN
-F 2 "zom:RFM95" H 6950 3900 30  0001 C CIN
-F 3 "" H 6950 3900 60  0000 C CNN
-	1    6950 3900
+P 7850 4050
+F 0 "U2" H 7500 4300 40  0000 C CNN
+F 1 "RFM95HW" H 8100 3300 40  0000 C CNN
+F 2 "zom:RFM95" H 7850 4050 30  0001 C CIN
+F 3 "" H 7850 4050 60  0000 C CNN
+	1    7850 4050
 	1    0    0    -1
 $EndComp
@@
 L GND #PWR07
 U 1 1 5B88846E
-P 6950 4850
-F 0 "#PWR07" H 6950 4600 50  0001 C CNN
-F 1 "GND" H 6950 4700 50  0000 C CNN
-F 2 "" H 6950 4850 50  0001 C CNN
-F 3 "" H 6950 4850 50  0001 C CNN
-	1    6950 4850
+P 7850 5000
+F 0 "#PWR07" H 7850 4750 50  0001 C CNN
+F 1 "GND" H 7850 4850 50  0000 C CNN
+F 2 "" H 7850 5000 50  0001 C CNN
+F 3 "" H 7850 5000 50  0001 C CNN
+	1    7850 5000
 	1    0    0    -1
 $EndComp
@@
 L Conn_01x01 J7
 U 1 1 5B88DC11
-P 6400 3550
-F 0 "J7" H 6400 3650 50  0000 C CNN
-F 1 "ANT" H 6400 3450 50  0000 C CNN
-F 2 "Pin_Headers:Pin_Header_Straight_1x01_Pitch2.54mm" H 6400 3550 50  0001 C CNN
-F 3 "" H 6400 3550 50  0001 C CNN
-	1    6400 3550
+P 7300 3700
+F 0 "J7" H 7300 3800 50  0000 C CNN
+F 1 "ANT" H 7300 3600 50  0000 C CNN
+F 2 "Pin_Headers:Pin_Header_Straight_1x01_Pitch2.54mm" H 7300 3700 50  0001 C CNN
+F 3 "" H 7300 3700 50  0001 C CNN
+	1    7300 3700
 	0    -1   -1   0
 $EndComp
@@
 L +3V3 #PWR024
 U 1 1 5B890347
-P 6950 3550
-F 0 "#PWR024" H 6950 3400 50  0001 C CNN
-F 1 "+3V3" H 6950 3690 50  0000 C CNN
-F 2 "" H 6950 3550 50  0001 C CNN
-F 3 "" H 6950 3550 50  0001 C CNN
-	1    6950 3550
+P 7850 3700
+F 0 "#PWR024" H 7850 3550 50  0001 C CNN
+F 1 "+3V3" H 7850 3840 50  0000 C CNN
+F 2 "" H 7850 3700 50  0001 C CNN
+F 3 "" H 7850 3700 50  0001 C CNN
+	1    7850 3700
 	1    0    0    -1
 $EndComp
@@
 L +3V3 #PWR025
 U 1 1 5B891AE7
-P 10500 2250
-F 0 "#PWR025" H 10500 2100 50  0001 C CNN
-F 1 "+3V3" H 10500 2390 50  0000 C CNN
-F 2 "" H 10500 2250 50  0001 C CNN
-F 3 "" H 10500 2250 50  0001 C CNN
-	1    10500 2250
+P 6350 3200
+F 0 "#PWR025" H 6350 3050 50  0001 C CNN
+F 1 "+3V3" H 6350 3340 50  0000 C CNN
+F 2 "" H 6350 3200 50  0001 C CNN
+F 3 "" H 6350 3200 50  0001 C CNN
+	1    6350 3200
 	1    0    0    -1
 $EndComp
@@
 Text Notes 6350 6600 0    60   ~ 0
 UART
-Text Notes 6850 3200 0    60   ~ 0
+Text Notes 8000 3400 0    60   ~ 0
 RFM95
 Text Notes 7200 5450 0    60   ~ 0
 DHT22
-Text Notes 8650 3550 0    60   ~ 0
+Text Notes 9550 3700 0    60   ~ 0
 RMF95 BREAKOUTS
 $Comp
 L Conn_01x12 J15
 U 1 1 5B90241E
-P 11100 1850
-F 0 "J15" H 11100 2450 50  0000 C CNN
-F 1 "misc" H 11100 1150 50  0000 C CNN
-F 2 "Pin_Headers:Pin_Header_Straight_1x12_Pitch2.54mm" H 11100 1850 50  0001 C CNN
-F 3 "" H 11100 1850 50  0001 C CNN
-	1    11100 1850
+P 6950 2800
+F 0 "J15" H 6950 3400 50  0000 C CNN
+F 1 "misc" H 6950 2100 50  0000 C CNN
+F 2 "Pin_Headers:Pin_Header_Straight_1x12_Pitch2.54mm" H 6950 2800 50  0001 C CNN
+F 3 "" H 6950 2800 50  0001 C CNN
+	1    6950 2800
 	1    0    0    -1
 $EndComp
@@
 	1    0    0    -1
 $EndComp
-Text GLabel 6400 3950 0    60   Input ~ 0
+Text GLabel 7300 4100 0    60   Input ~ 0
 26
-Text GLabel 6400 4050 0    60   Input ~ 0
+Text GLabel 7300 4200 0    60   Input ~ 0
 33
-Text GLabel 6400 4150 0    60   Input ~ 0
+Text GLabel 7300 4300 0    60   Input ~ 0
 32
-Text GLabel 6400 4250 0    60   Input ~ 0
+Text GLabel 7300 4400 0    60   Input ~ 0
 25
-Text GLabel 6400 4450 0    60   Input ~ 0
+Text GLabel 7300 4600 0    60   Input ~ 0
 27
 Text GLabel 5300 2400 2    60   Input ~ 0
 TX0
-Text GLabel 5300 2300 2    60   Input ~ 0
-22
 Text GLabel 5300 2600 2    60   Input ~ 0
 21
@@
 	1    0    0    -1
 $EndComp
-Text GLabel 7500 4400 2    60   Input ~ 0
+Text GLabel 8400 4550 2    60   Input ~ 0
 DIO5
 $Comp
 L Conn_01x06 J10
 U 1 1 5B91954E
-P 8800 4100
-F 0 "J10" H 8800 4400 50  0000 C CNN
-F 1 "LBD" H 8800 3700 50  0000 C CNN
-F 2 "Pin_Headers:Pin_Header_Straight_1x06_Pitch2.54mm" H 8800 4100 50  0001 C CNN
-F 3 "" H 8800 4100 50  0001 C CNN
-	1    8800 4100
-	1    0    0    -1
-$EndComp
-Text GLabel 7500 4300 2    60   Input ~ 0
+P 9700 4250
+F 0 "J10" H 9700 4550 50  0000 C CNN
+F 1 "LBD" H 9700 3850 50  0000 C CNN
+F 2 "Pin_Headers:Pin_Header_Straight_1x06_Pitch2.54mm" H 9700 4250 50  0001 C CNN
+F 3 "" H 9700 4250 50  0001 C CNN
+	1    9700 4250
+	1    0    0    -1
+$EndComp
+Text GLabel 8400 4450 2    60   Input ~ 0
 DIO4
-Text GLabel 7500 4200 2    60   Input ~ 0
+Text GLabel 8400 4350 2    60   Input ~ 0
 DIO3
-Text GLabel 7500 4100 2    60   Input ~ 0
+Text GLabel 8400 4250 2    60   Input ~ 0
 DIO2
-Text GLabel 7500 4000 2    60   Input ~ 0
+Text GLabel 8400 4150 2    60   Input ~ 0
 DIO1
-Text GLabel 7500 3900 2    60   Input ~ 0
+Text GLabel 8400 4050 2    60   Input ~ 0
 DIO0
-Text GLabel 8600 3900 0    60   Input ~ 0
+Text GLabel 9500 4050 0    60   Input ~ 0
 DIO2
-Text GLabel 8600 4000 0    60   Input ~ 0
+Text GLabel 9500 4150 0    60   Input ~ 0
 DIO1
-Text GLabel 8600 4100 0    60   Input ~ 0
+Text GLabel 9500 4250 0    60   Input ~ 0
 DIO0
 $Comp
 L +3V3 #PWR036
 U 1 1 5B91A050
-P 8100 4200
-F 0 "#PWR036" H 8100 4050 50  0001 C CNN
-F 1 "+3V3" H 8100 4340 50  0000 C CNN
-F 2 "" H 8100 4200 50  0001 C CNN
-F 3 "" H 8100 4200 50  0001 C CNN
-	1    8100 4200
-	1    0    0    -1
-$EndComp
-Text GLabel 8600 4300 0    60   Input ~ 0
+P 9000 4350
+F 0 "#PWR036" H 9000 4200 50  0001 C CNN
+F 1 "+3V3" H 9000 4490 50  0000 C CNN
+F 2 "" H 9000 4350 50  0001 C CNN
+F 3 "" H 9000 4350 50  0001 C CNN
+	1    9000 4350
+	1    0    0    -1
+$EndComp
+Text GLabel 9500 4450 0    60   Input ~ 0
 DIO4
-Text GLabel 8600 4400 0    60   Input ~ 0
+Text GLabel 9500 4550 0    60   Input ~ 0
 DIO3
 $Comp
 L Conn_02x03_Odd_Even J16
 U 1 1 5B91ABB9
-P 9500 4250
-F 0 "J16" H 9550 4450 50  0000 C CNN
-F 1 "LBO" H 9550 4050 50  0000 C CNN
-F 2 "Pin_Headers:Pin_Header_Straight_2x03_Pitch2.54mm" H 9500 4250 50  0001 C CNN
-F 3 "" H 9500 4250 50  0001 C CNN
-	1    9500 4250
+P 10400 4400
+F 0 "J16" H 10450 4600 50  0000 C CNN
+F 1 "LBO" H 10450 4200 50  0000 C CNN
+F 2 "Pin_Headers:Pin_Header_Straight_2x03_Pitch2.54mm" H 10400 4400 50  0001 C CNN
+F 3 "" H 10400 4400 50  0001 C CNN
+	1    10400 4400
 	0    -1   -1   0
 $EndComp
-Text GLabel 9400 3950 1    60   Input ~ 0
+Text GLabel 10300 4100 1    60   Input ~ 0
 32
-Text GLabel 9500 3950 1    60   Input ~ 0
+Text GLabel 10400 4100 1    60   Input ~ 0
 25
-Text GLabel 9600 3950 1    60   Input ~ 0
+Text GLabel 10500 4100 1    60   Input ~ 0
 27
-Text GLabel 9400 4450 3    60   Input ~ 0
+Text GLabel 10300 4600 3    60   Input ~ 0
 33
-Text GLabel 9500 4450 3    60   Input ~ 0
+Text GLabel 10400 4600 3    60   Input ~ 0
 26
-Text GLabel 9600 4450 3    60   Input ~ 0
+Text GLabel 10500 4600 3    60   Input ~ 0
 DIO5
 Text GLabel 9200 1500 0    60   Input ~ 0
@@
 L GND #PWR037
 U 1 1 5B891B40
-P 10200 2150
-F 0 "#PWR037" H 10200 1900 50  0001 C CNN
-F 1 "GND" H 10200 2000 50  0000 C CNN
-F 2 "" H 10200 2150 50  0001 C CNN
-F 3 "" H 10200 2150 50  0001 C CNN
-	1    10200 2150
+P 6050 3100
+F 0 "#PWR037" H 6050 2850 50  0001 C CNN
+F 1 "GND" H 6050 2950 50  0000 C CNN
+F 2 "" H 6050 3100 50  0001 C CNN
+F 3 "" H 6050 3100 50  0001 C CNN
+	1    6050 3100
 	1    0    0    -1
 $EndComp
@@
 	5300 6750 4800 6750
 Wire Wire Line
-	8100 4200 8600 4200
+	9000 4350 9500 4350
 Wire Wire Line
 	4150 7050 4150 7250
@@
 	1950 3350 1950 3400
 Wire Wire Line
-	6950 4750 6950 4850
-Connection ~ 6950 4850
-Wire Wire Line
-	7050 4850 7050 4750
-Wire Wire Line
-	6850 4850 7050 4850
-Wire Wire Line
-	6850 4750 6850 4850
+	7850 4900 7850 5000
+Connection ~ 7850 5000
+Wire Wire Line
+	7950 5000 7950 4900
+Wire Wire Line
+	7750 5000 7950 5000
+Wire Wire Line
+	7750 4900 7750 5000
 Connection ~ 5400 3600
 Wire Wire Line
@@
 Text GLabel 6550 7100 0    60   Input ~ 0
 19
-Text GLabel 10900 2350 0    60   Input ~ 0
+Text GLabel 6750 3300 0    60   Input ~ 0
 14/SCL
-Text GLabel 10900 2450 0    60   Input ~ 0
+Text GLabel 6750 3400 0    60   Input ~ 0
 12/SDA
 Wire Wire Line
-	10900 2250 10500 2250
-Wire Wire Line
-	10900 2150 10200 2150
+	6750 3200 6350 3200
+Wire Wire Line
+	6750 3100 6050 3100
+Text GLabel 6750 2500 0    60   Input ~ 0
+21
+Text GLabel 6750 2600 0    60   Input ~ 0
+19
+Text GLabel 6750 2800 0    60   Input ~ 0
+2
+Text GLabel 6750 2400 0    60   Input ~ 0
+35
+Text GLabel 6750 2700 0    60   Input ~ 0
+5
+Text GLabel 6750 2900 0    60   Input ~ 0
+0
+Text GLabel 6750 3000 0    60   Input ~ 0
+VIN
+$Comp
+L +5V #PWR038
+U 1 1 5B927367
+P 6750 2300
+F 0 "#PWR038" H 6750 2150 50  0001 C CNN
+F 1 "+5V" H 6750 2440 50  0000 C CNN
+F 2 "" H 6750 2300 50  0001 C CNN
+F 3 "" H 6750 2300 50  0001 C CNN
+	1    6750 2300
+	1    0    0    -1
+$EndComp
+Text GLabel 5300 2300 2    60   Input ~ 0
+22
 $EndSCHEMATC

Commit message: update
Connections:
- net +3V3: now also J5.4 (Pin_4); no longer J5.3 (Pin_3)
- net GND: now also J5.3 (Pin_3); no longer J5.4 (Pin_4)
- no-connect marks 0 -> 3
Changed lines of the file:
@@
 L GND #PWR015
 U 1 1 5B88CAD4
-P 4700 5750
-F 0 "#PWR015" H 4700 5500 50  0001 C CNN
-F 1 "GND" H 4700 5600 50  0000 C CNN
-F 2 "" H 4700 5750 50  0001 C CNN
-F 3 "" H 4700 5750 50  0001 C CNN
-	1    4700 5750
+P 4750 5650
+F 0 "#PWR015" H 4750 5400 50  0001 C CNN
+F 1 "GND" H 4750 5500 50  0000 C CNN
+F 2 "" H 4750 5650 50  0001 C CNN
+F 3 "" H 4750 5650 50  0001 C CNN
+	1    4750 5650
 	1    0    0    -1
 $EndComp
@@
 L +3V3 #PWR016
 U 1 1 5B88CCC7
-P 4450 5650
-F 0 "#PWR016" H 4450 5500 50  0001 C CNN
-F 1 "+3V3" H 4450 5790 50  0000 C CNN
-F 2 "" H 4450 5650 50  0001 C CNN
-F 3 "" H 4450 5650 50  0001 C CNN
-	1    4450 5650
+P 4450 5900
+F 0 "#PWR016" H 4450 5750 50  0001 C CNN
+F 1 "+3V3" H 4450 6040 50  0000 C CNN
+F 2 "" H 4450 5900 50  0001 C CNN
+F 3 "" H 4450 5900 50  0001 C CNN
+	1    4450 5900
 	1    0    0    -1
 $EndComp
@@
 	7500 6050 7400 6050
 Wire Wire Line
-	4450 5650 4900 5650
-Wire Wire Line
-	4700 5750 4900 5750
-Wire Wire Line
 	3200 5750 3550 5750
 Wire Wire Line
@@
 Text GLabel 5300 2300 2    60   Input ~ 0
 22
+NoConn ~ 6050 1250
+NoConn ~ 5900 4800
+NoConn ~ 3100 5900
+Wire Wire Line
+	4900 5650 4750 5650
+Wire Wire Line
+	4900 5900 4900 5750
+Wire Wire Line
+	4450 5900 4900 5900
 $EndSCHEMATC

Commit message: update
Connections:
- net +3V3: now also J1.3 (Pin_3); no longer J1.1 (Pin_1)
- net +5V: now also J6.3 (Pin_3); no longer J6.1 (Pin_1)
- net VIN: now also J6.1 (Pin_1); no longer J6.3 (Pin_3)
- net at C1.1, D1.1 (K), D2.1 (K): now also J1.1 (Pin_1); no longer J1.3 (Pin_3)
Other:
- moved on the sheet: J1, J6
Changed lines of the file:
@@
 F 3 "" H 1000 1350 50  0001 C CNN
 	1    1000 1350
-	-1   0    0    1
+	1    0    0    -1
 $EndComp
 Text Notes 950  900  0    60   ~ 0
@@
 F 3 "" H 6100 1450 50  0001 C CNN
 	1    6100 1450
-	-1   0    0    1
+	1    0    0    -1
 $EndComp
 Text Notes 6050 1000 0    60   ~ 0
@@
 	6300 1350 6300 1150
 Wire Wire Line
-	6300 1450 6900 1450
+	5900 1450 6900 1450
 Connection ~ 7100 6050
 Wire Wire Line
@@
 	1200 1250 1200 1050
 Wire Wire Line
-	1200 1350 1800 1350
+	800  1350 1800 1350
 Wire Wire Line
 	6000 5400 6000 5600
@@
 Wire Wire Line
 	4450 5900 4900 5900
+Wire Wire Line
+	1200 1250 800  1250
+Wire Wire Line
+	1200 1450 800  1450
+Wire Wire Line
+	6300 1350 5900 1350
+Wire Wire Line
+	6300 1550 5900 1550
 $EndSCHEMATC

Commit message: update
Parts:
- C3, C4: value C -> 1uF
- R2, R3: value R -> 10K
- R5, R6, R7: value R -> 4.7K
Changed lines of the file:
@@
 P 1500 3000
 F 0 "R2" V 1580 3000 50  0000 C CNN
-F 1 "R" V 1500 3000 50  0000 C CNN
+F 1 "10K" V 1500 3000 50  0000 C CNN
 F 2 "Resistors_THT:R_Axial_DIN0204_L3.6mm_D1.6mm_P1.90mm_Vertical" V 1430 3000 50  0001 C CNN
 F 3 "" H 1500 3000 50  0001 C CNN
@@
 P 1500 3600
 F 0 "R3" V 1580 3600 50  0000 C CNN
-F 1 "R" V 1500 3600 50  0000 C CNN
+F 1 "10K" V 1500 3600 50  0000 C CNN
 F 2 "Resistors_THT:R_Axial_DIN0204_L3.6mm_D1.6mm_P1.90mm_Vertical" V 1430 3600 50  0001 C CNN
 F 3 "" H 1500 3600 50  0001 C CNN
@@
 P 1300 6900
 F 0 "C3" H 1325 7000 50  0000 L CNN
-F 1 "C" H 1325 6800 50  0000 L CNN
+F 1 "1uF" H 1325 6800 50  0000 L CNN
 F 2 "Capacitors_THT:C_Disc_D3.0mm_W1.6mm_P2.50mm" H 1338 6750 50  0001 C CNN
 F 3 "" H 1300 6900 50  0001 C CNN
@@
 P 2250 6900
 F 0 "C4" H 2275 7000 50  0000 L CNN
-F 1 "C" H 2275 6800 50  0000 L CNN
+F 1 "1uF" H 2275 6800 50  0000 L CNN
 F 2 "Capacitors_THT:C_Disc_D3.0mm_W1.6mm_P2.50mm" H 2288 6750 50  0001 C CNN
 F 3 "" H 2250 6900 50  0001 C CNN
@@
 P 7100 5900
 F 0 "R7" V 7180 5900 50  0000 C CNN
-F 1 "R" V 7100 5900 50  0000 C CNN
+F 1 "4.7K" V 7100 5900 50  0000 C CNN
 F 2 "Resistors_THT:R_Axial_DIN0204_L3.6mm_D1.6mm_P1.90mm_Vertical" V 7030 5900 50  0001 C CNN
 F 3 "" H 7100 5900 50  0001 C CNN
@@
 P 3800 6900
 F 0 "R5" V 3880 6900 50  0000 C CNN
-F 1 "R" V 3800 6900 50  0000 C CNN
+F 1 "4.7K" V 3800 6900 50  0000 C CNN
 F 2 "Resistors_THT:R_Axial_DIN0204_L3.6mm_D1.6mm_P1.90mm_Vertical" V 3730 6900 50  0001 C CNN
 F 3 "" H 3800 6900 50  0001 C CNN
@@
 P 4150 6900
 F 0 "R6" V 4230 6900 50  0000 C CNN
-F 1 "R" V 4150 6900 50  0000 C CNN
+F 1 "4.7K" V 4150 6900 50  0000 C CNN
 F 2 "Resistors_THT:R_Axial_DIN0204_L3.6mm_D1.6mm_P1.90mm_Vertical" V 4080 6900 50  0001 C CNN
 F 3 "" H 4150 6900 50  0001 C CNN
