File: hardware/zom/zom1a.kicad_pcb (KiCad board)
At the start: 2 copper layers, 51.5 x 76.2 mm, 37 parts, among them J1 REG:3V3, J10 LBD, J11 uart, J12 dht22, J13 9602-a, J14 satx, J15 misc, J16 LBO, J19 9602-b, J2 prog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

Commit message: update
Parts:
- removed R8: R, Resistors_THT:R_Axial_DIN0204_L3.6mm_D1.6mm_P1.90mm_Vertical
- added J17: VIN2, Pin_Headers:Pin_Header_Straight_1x02_Pitch2.54mm, F.Cu at (58.4, 64.1)
- moved Q2 54.2 mm to (48.3, 52.1), turned to 0 degrees
- moved Q1 46.0 mm to (57.8, 46.4)
- moved R3 46.0 mm to (48.9, 45.1)
- moved R2 39.1 mm to (56.5, 52.7), turned to 180 degrees
- moved R5 34.0 mm to (63.5, 58.4), turned to 90 degrees
- moved R6 34.0 mm to (59.1, 58.4), turned to 90 degrees
- moved R7 33.4 mm to (103.5, 80.0)
- moved J12 23.0 mm to (109.9, 80.0)
- moved SW2 7.41 mm to (108.0, 63.5), turned to 0 degrees
- moved J5 3.42 mm to (97.2, 59.1)
- moved C3 3.24 mm to (103.5, 71.1), turned to 180 degrees
- moved R1 2.84 mm to (101.6, 75.6), turned to 0 degrees
- moved C4 1.42 mm to (101.0, 63.5)
- moved C6 1.27 mm to (110.5, 91.4)
- moved R4 0.90 mm to (101.6, 67.3)
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Connections:
- net 34 renamed 34/RX1
- net DIO1 renamed Net-(J10-Pad2)
- net DIO4 renamed Net-(J10-Pad5)
- C1 pad 2: GND -> Net-(C1-Pad2)
- C2 pad 1: GND -> Net-(C1-Pad2)
- C2 pad 2: +3V3 -> 22
- C5 pad 2: GND -> Net-(C5-Pad2)
- C6 pad 1: GND -> Net-(C5-Pad2)
- J1 pad 1: +3V3 -> 22
- J10 pad 1: DIO2 -> Net-(J10-Pad1)
- J10 pad 3: DIO0 -> Net-(J10-Pad3)
- J10 pad 4: +3V3 -> Net-(J10-Pad4)
- J10 pad 6: DIO3 -> Net-(J10-Pad6)
- J11 pad 1: +3V3 -> 33/TX2
- J11 pad 2: VIN -> 35/RX2
- J11 pad 3: (no net) -> 22
- J11 pad 4: (no net) -> VIN
- J12 pad 1: +3V3 -> 22
- J12 pad 2: Net-(J12-Pad2) -> 25
- J13 pad 3: 13 -> 32/TX1
- J15 pad 10: (no net) -> 33/TX2
- J15 pad 11: (no net) -> 35/RX2
- J15 pad 2: +3V3 -> 22
- J15 pad 4: (no net) -> SCL
- J15 pad 5: (no net) -> SDA
- J15 pad 6: (no net) -> 0
- J15 pad 7: (no net) -> 2
- J15 pad 8: (no net) -> 13
- J15 pad 9: (no net) -> 26
- J16 pad 1: 33 -> 12
- J16 pad 2: 32 -> 5
- J16 pad 3: 26 -> 18
- J16 pad 4: 25 -> 15
- J16 pad 5: DIO5 -> 19
- J16 pad 6: 27 -> GND
- J2 pad 4: RXD0 -> (no net)
- J2 pad 5: TXD0 -> (no net)
- J4 pad 1: (no net) -> 14
- J4 pad 2: (no net) -> 21
- J4 pad 4: +3V3 -> 22
- J4 pad 5: (no net) -> 23
- J4 pad 7: (no net) -> 17
- J5 pad 1: 12/SDA -> SDA
- J5 pad 2: 14/SCL -> SCL
- J5 pad 3: +3V3 -> 22
- J8 pad 1: +3V3 -> SDA
- J8 pad 2: GND -> SCL
- J8 pad 3: 12/SDA -> 22
- J8 pad 4: 14/SCL -> GND
- J9 pad 1: GND -> 22
- J9 pad 2: Net-(J9-Pad2) -> 22
- J9 pad 3: +3V3 -> GND
- R1 pad 1: +3V3 -> 22
- R4 pad 1: +3V3 -> 22
- R5 pad 1: +3V3 -> 22
- R5 pad 2: 12/SDA -> SCL
- R6 pad 1: +3V3 -> 22
- R6 pad 2: 14/SCL -> SDA
- R7 pad 1: +3V3 -> 22
- R7 pad 2: Net-(J12-Pad2) -> 25
- U1 pad 12: 27 -> 27/SAT_SLEEP
- U1 pad 13: 14/SCL -> 14
- U1 pad 14: 12/SDA -> 12
- U1 pad 2: +3V3 -> 22
- U1 pad 23: (no net) -> 15
- U1 pad 24: (no net) -> 2
- U1 pad 26: (no net) -> SDA
- U1 pad 27: (no net) -> SCL
- U1 pad 28: (no net) -> 17
- U1 pad 29: (no net) -> 5
- U1 pad 30: (no net) -> 18
- U1 pad 31: (no net) -> 19
- U1 pad 33: (no net) -> 21
- U1 pad 34: RXD0 -> (no net)
- U1 pad 35: TXD0 -> (no net)
- U1 pad 36: (no net) -> 22
- U1 pad 37: (no net) -> 23
- U1 pad 7: (no net) -> 35/RX2
- U1 pad 8: 32 -> 32/TX1
- U1 pad 9: 33 -> 33/TX2
- U2 pad 11: DIO3 -> Net-(J10-Pad4)
- U2 pad 13: +3V3 -> 22
- U2 pad 14: DIO0 -> Net-(J10-Pad1)
- U2 pad 16: DIO2 -> Net-(J10-Pad3)
- U2 pad 2: 32 -> 19
- U2 pad 3: 33 -> 18
- U2 pad 4: 25 -> 5
- U2 pad 5: 26 -> 12
- U2 pad 6: 27 -> 15
- U2 pad 7: DIO5 -> Net-(J10-Pad6)
Routing:
- net GND: track 208.0 -> 24.7 mm, vias 3 -> 0
- net +3V3: track 141.3 -> 0.00 mm, vias 3 -> 0
- net 13: track 44.4 -> 0.00 mm, vias 1 -> 0
- net VIN: track 44.2 -> 0.00 mm
- net 18: track 0.00 -> 40.2 mm, vias 0 -> 2
- net 34/RX1: track 39.1 -> 0.00 mm, vias 1 -> 0
- net 14/SCL: track 38.9 -> 0.00 mm, vias 1 -> 0
- net DTR: track 38.2 -> 0.00 mm
- net 33: track 36.9 -> 0.00 mm
- net 12/SDA: track 36.3 -> 0.00 mm
- net 32: track 36.0 -> 0.00 mm
- net 26: track 31.1 -> 0.00 mm
- net 25: track 30.9 -> 0.00 mm
- net 0: track 30.2 -> 0.00 mm
- net RTS: track 29.8 -> 0.00 mm, vias 1 -> 0
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Other:
- net class power removed
