File: hardware/zom/zom2.kicad_pcb (KiCad board)
At the start: 2 copper layers, 51.5 x 76.2 mm, 37 parts, among them J1 REG:3V3, J10 LBD, J11 uart, J12 dht22, J13 9602-a, J14 satx, J15 misc, J16 LBO, J19 9602-b, J2 prog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

Commit message: update
Parts:
- moved J12 25.9 mm to (132.7, 77.5), turned to 0 degrees
- moved R7 18.8 mm to (134.6, 67.9)
- moved R8 13.1 mm to (100.3, 89.5)
- moved C4 4.07 mm to (101.6, 64.8), turned to 0 degrees
Connections:
- net RX0 renamed RXD0
- net TX0 renamed TXD0
- J12 pad 2: 18 -> Net-(J12-Pad2)
- J14 pad 3: 23/SAT_SLEEP -> 27/SAT_SLEEP
- J15 pad 1: 35 -> VIN
- J15 pad 11: VIN -> (no net)
- J15 pad 12: (no net) -> 27/SAT_SLEEP
- J15 pad 4: 23/SAT_SLEEP -> (no net)
- J19 pad 6: 23/SAT_SLEEP -> 27/SAT_SLEEP
- J4 pad 1: 15 -> (no net)
- J4 pad 2: 4 -> (no net)
- J4 pad 5: 16 -> (no net)
- J4 pad 7: 17 -> (no net)
- R7 pad 2: 18 -> Net-(J12-Pad2)
- U1 pad 23: 15 -> (no net)
- U1 pad 26: 4 -> (no net)
- U1 pad 27: 16 -> (no net)
- U1 pad 28: 17 -> (no net)
- U1 pad 30: 18 -> (no net)
- U1 pad 33: 23/SAT_SLEEP -> (no net)
- U1 pad 7: 35 -> (no net)
Routing:
- net 23/SAT_SLEEP: track 79.4 -> 0.00 mm, vias 2 -> 0
- net 4: track 78.3 -> 0.00 mm, vias 1 -> 0
- net 17: track 76.2 -> 0.00 mm, vias 1 -> 0
- net 16: track 76.0 -> 0.00 mm, vias 1 -> 0
- net 15: track 73.3 -> 0.00 mm, vias 1 -> 0
- net GND: track 256.5 -> 214.3 mm, vias 5 -> 3
- net +5V: track 44.0 -> 10.2 mm, vias 1 -> 0
- net 35: track 28.9 -> 0.00 mm, vias 2 -> 0
- net 18: track 22.6 -> 0.00 mm, vias 1 -> 0
- net +3V3: track 169.2 -> 149.1 mm
- net 14/SCL: track 21.4 -> 38.9 mm, vias 0 -> 1
- net Net-(J9-Pad2): track 11.2 -> 0.00 mm
- net 13: track 53.4 -> 44.4 mm
- net 0: track 36.7 -> 30.2 mm, vias 1 -> 0
- net 27/SAT_SLEEP: track 0.00 -> 4.30 mm
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