File: hardware/zom/zom2.sch (KiCad schematic (older format))
At the start: 37 parts, among them J1 REG:3V3, J10 LBD, J11 uart, J12 dht22, J13 9602-a, J14 satx, J15 misc, J16 LBO, J19 9602-b, J2 prog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

Commit message: update
Connections:
- net labels added: 21, 27/SAT_SLEEP, RXD0, TXD0
- net labels removed: 23/SAT_SLEEP, RX0, TX0
Changed lines of the file:
@@
 0
 Text GLabel 5300 2600 2    60   Input ~ 0
-23/SAT_SLEEP
+21
 Text GLabel 5300 2500 2    60   Input ~ 0
-RX0
+RXD0
 $Comp
 L GND #PWR04
@@
 Text GLabel 1350 5150 0    60   Input ~ 0
 RTS
+Text GLabel 1350 5050 0    60   Input ~ 0
+TXD0
+Text GLabel 1350 4950 0    60   Input ~ 0
+RXD0
 Text GLabel 1350 4850 0    60   Input ~ 0
 VIN
@@
 $EndComp
 $Comp
+L GND #PWR026
+U 1 1 5B891B40
+P 10600 1550
+F 0 "#PWR026" H 10600 1300 50  0001 C CNN
+F 1 "GND" H 10600 1400 50  0000 C CNN
+F 2 "" H 10600 1550 50  0001 C CNN
+F 3 "" H 10600 1550 50  0001 C CNN
+	1    10600 1550
+	1    0    0    -1
+$EndComp
+Text GLabel 10900 1350 0    60   Input ~ 0
+VIN
+$Comp
 L Conn_01x02 J3
 U 1 1 5B89258D
@@
 VIN
 $Comp
-L GND #PWR026
+L GND #PWR027
 U 1 1 5B89266B
 P 2900 1200
-F 0 "#PWR026" H 2900 950 50  0001 C CNN
+F 0 "#PWR027" H 2900 950 50  0001 C CNN
 F 1 "GND" H 2900 1050 50  0000 C CNN
 F 2 "" H 2900 1200 50  0001 C CNN
@@
 $EndComp
 $Comp
-L +3V3 #PWR027
+L +3V3 #PWR028
 U 1 1 5B892FAF
 P 4150 6750
-F 0 "#PWR027" H 4150 6600 50  0001 C CNN
+F 0 "#PWR028" H 4150 6600 50  0001 C CNN
 F 1 "+3V3" H 4150 6890 50  0000 C CNN
 F 2 "" H 4150 6750 50  0001 C CNN
@@
 VIN
 $Comp
-L GND #PWR028
+L GND #PWR029
 U 1 1 5B895E60
 P 6900 1450
-F 0 "#PWR028" H 6900 1200 50  0001 C CNN
+F 0 "#PWR029" H 6900 1200 50  0001 C CNN
 F 1 "GND" H 6900 1300 50  0000 C CNN
 F 2 "" H 6900 1450 50  0001 C CNN
@@
 $EndComp
 $Comp
-L GND #PWR029
+L GND #PWR030
 U 1 1 5B8973E2
 P 8650 1900
-F 0 "#PWR029" H 8650 1650 50  0001 C CNN
+F 0 "#PWR030" H 8650 1650 50  0001 C CNN
 F 1 "GND" H 8650 1750 50  0000 C CNN
 F 2 "" H 8650 1900 50  0001 C CNN
@@
 $EndComp
 $Comp
-L +5V #PWR030
+L +5V #PWR031
 U 1 1 5B897541
 P 7150 1750
-F 0 "#PWR030" H 7150 1600 50  0001 C CNN
+F 0 "#PWR031" H 7150 1600 50  0001 C CNN
 F 1 "+5V" H 7150 1890 50  0000 C CNN
 F 2 "" H 7150 1750 50  0001 C CNN
@@
 $EndComp
 $Comp
-L +5V #PWR031
+L +5V #PWR032
 U 1 1 5B89761E
 P 8400 2200
-F 0 "#PWR031" H 8400 2050 50  0001 C CNN
+F 0 "#PWR032" H 8400 2050 50  0001 C CNN
 F 1 "+5V" H 8400 2340 50  0000 C CNN
 F 2 "" H 8400 2200 50  0001 C CNN
@@
 $EndComp
 $Comp
-L GND #PWR032
+L GND #PWR033
 U 1 1 5B897911
 P 9200 2800
-F 0 "#PWR032" H 9200 2550 50  0001 C CNN
+F 0 "#PWR033" H 9200 2550 50  0001 C CNN
 F 1 "GND" H 9200 2650 50  0000 C CNN
 F 2 "" H 9200 2800 50  0001 C CNN
@@
 Iridium 9602
 Text GLabel 9200 2600 0    60   Input ~ 0
-23/SAT_SLEEP
-$Comp
-L +5V #PWR033
+27/SAT_SLEEP
+$Comp
+L +5V #PWR034
 U 1 1 5B899DD3
 P 8400 1700
-F 0 "#PWR033" H 8400 1550 50  0001 C CNN
+F 0 "#PWR034" H 8400 1550 50  0001 C CNN
 F 1 "+5V" H 8400 1840 50  0000 C CNN
 F 2 "" H 8400 1700 50  0001 C CNN
@@
 SAT_LION
 $Comp
-L +3V3 #PWR034
+L +3V3 #PWR035
 U 1 1 5B89AA80
 P 6550 6800
-F 0 "#PWR034" H 6550 6650 50  0001 C CNN
+F 0 "#PWR035" H 6550 6650 50  0001 C CNN
 F 1 "+3V3" H 6550 6940 50  0000 C CNN
 F 2 "" H 6550 6800 50  0001 C CNN
@@
 	1    0    0    -1
 $EndComp
-Text GLabel 10900 1650 0    60   Input ~ 0
-23/SAT_SLEEP
+Text GLabel 10900 2450 0    60   Input ~ 0
+27/SAT_SLEEP
 Text Notes 7200 5450 0    60   ~ 0
 DHT22
@@
 $EndComp
 $Comp
-L GND #PWR035
+L GND #PWR036
 U 1 1 5B902A1C
 P 6550 7200
-F 0 "#PWR035" H 6550 6950 50  0001 C CNN
+F 0 "#PWR036" H 6550 6950 50  0001 C CNN
 F 1 "GND" H 6550 7050 50  0000 C CNN
 F 2 "" H 6550 7200 50  0001 C CNN
@@
 27
 Text GLabel 5300 2400 2    60   Input ~ 0
-TX0
+TXD0
 Text GLabel 5300 2300 2    60   Input ~ 0
 22
@@
 DIO0
 $Comp
-L +3V3 #PWR036
+L +3V3 #PWR037
 U 1 1 5B91A050
 P 8100 4200
-F 0 "#PWR036" H 8100 4050 50  0001 C CNN
+F 0 "#PWR037" H 8100 4050 50  0001 C CNN
 F 1 "+3V3" H 8100 4340 50  0000 C CNN
 F 2 "" H 8100 4200 50  0001 C CNN
@@
 Text GLabel 4150 7250 3    60   Input ~ 0
 14/SCL
-Text GLabel 3550 5850 0    60   Input ~ 0
-17
-Text GLabel 3550 5650 0    60   Input ~ 0
-16
-Text GLabel 3550 5350 0    60   Input ~ 0
-4
-Text GLabel 3550 5250 0    60   Input ~ 0
-15
-Text GLabel 10900 1350 0    60   Input ~ 0
-35
-Text GLabel 10900 2350 0    60   Input ~ 0
-VIN
-Text GLabel 6900 6050 0    60   Input ~ 0
-18
-$Comp
-L GND #PWR037
-U 1 1 5B891B40
-P 10600 1550
-F 0 "#PWR037" H 10600 1300 50  0001 C CNN
-F 1 "GND" H 10600 1400 50  0000 C CNN
-F 2 "" H 10600 1550 50  0001 C CNN
-F 3 "" H 10600 1550 50  0001 C CNN
-	1    10600 1550
-	1    0    0    -1
-$EndComp
-Text GLabel 1350 5050 0    60   Input ~ 0
-TX0
-Text GLabel 1350 4950 0    60   Input ~ 0
-RX0
 Wire Wire Line
 	5850 5400 6000 5400
@@
 Wire Wire Line
 	10500 1450 10900 1450
+Wire Wire Line
+	10900 1550 10600 1550
 Connection ~ 7100 6050
 Wire Wire Line
@@
 Connection ~ 1400 1350
 Connection ~ 2950 -750
-Wire Wire Line
-	10900 1550 10600 1550
 $EndSCHEMATC
