File: hardware/zom/zom3.kicad_pcb (KiCad board)
At the start: 2 copper layers, 51.6 x 75.9 mm, 39 parts, among them J1 REG:3V3, J10 LBD, J11 uart, J12 dht22, J13 9602-a, J14 satx, J15 misc, J16 LBO, J19 9602-b, J2 prog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

Commit message: update
Other:
- board size 51.6 x 75.9 mm -> 51.5 x 76.2 mm
Changed lines of the file:
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@@
     (links 127)
     (no_connects 0)
-    (area 72.924599 30.404999 124.636601 106.501001)
+    (area 72.949999 30.404999 124.610001 106.755001)
     (thickness 1.6)
-    (drawings 25)
+    (drawings 17)
     (tracks 697)
     (zones 0)
@@
     )
   )
-  (gr_line (start 73.0504 106.426) (end 124.5616 106.426) (angle 90) (layer Edge.Cuts) (width 0.15))
-  (gr_line (start 72.9996 106.426) (end 73.914 106.426) (angle 90) (layer Edge.Cuts) (width 0.15))
-  (gr_line (start 72.9996 30.48) (end 72.9996 106.426) (angle 90) (layer Edge.Cuts) (width 0.15))
-  (gr_line (start 124.5616 30.48) (end 72.9996 30.48) (angle 90) (layer Edge.Cuts) (width 0.15))
-  (gr_line (start 124.5616 106.426) (end 124.5616 30.48) (angle 90) (layer Edge.Cuts) (width 0.15))
-  (gr_line (start 72.9996 30.7848) (end 73.0504 30.7848) (angle 90) (layer Dwgs.User) (width 0.2))
-  (gr_line (start 72.9996 30.48) (end 72.9996 30.7848) (angle 90) (layer Dwgs.User) (width 0.2))
-  (gr_line (start 73.406 30.48) (end 72.9996 30.48) (angle 90) (layer Dwgs.User) (width 0.2))
-  (gr_line (start 124.5616 30.7848) (end 124.5108 30.7848) (angle 90) (layer Dwgs.User) (width 0.2))
-  (gr_line (start 124.5616 30.48) (end 124.5616 30.7848) (angle 90) (layer Dwgs.User) (width 0.2))
-  (gr_line (start 124.2568 30.48) (end 124.5616 30.48) (angle 90) (layer Dwgs.User) (width 0.2))
-  (gr_line (start 124.5235 106.4895) (end 124.5235 106.2355) (angle 90) (layer Dwgs.User) (width 0.2))
-  (gr_line (start 124.2695 106.4895) (end 124.5235 106.4895) (angle 90) (layer Dwgs.User) (width 0.2))
   (gr_line (start 76.2 81.915) (end 76.2 84.455) (angle 90) (layer Dwgs.User) (width 0.2))
   (gr_line (start 76.2 80.01) (end 76.2 81.915) (angle 90) (layer Dwgs.User) (width 0.2))
+  (gr_circle (center 75 104.775) (end 76.2 105.41) (layer Edge.Cuts) (width 0.15))
+  (gr_line (start 73.025 106.68) (end 73.025 30.48) (angle 90) (layer Edge.Cuts) (width 0.15))
+  (gr_line (start 124.535 106.48) (end 73.025 106.48) (angle 90) (layer Edge.Cuts) (width 0.15))
+  (gr_line (start 124.535 30.48) (end 124.535 106.48) (angle 90) (layer Edge.Cuts) (width 0.15))
+  (gr_line (start 73.025 30.48) (end 124.46 30.48) (angle 90) (layer Edge.Cuts) (width 0.15))
   (gr_line (start 76.2 83.1) (end 74.93 83.1) (angle 90) (layer Dwgs.User) (width 0.2))
   (gr_line (start 77.47 66.23) (end 72.39 66.23) (angle 90) (layer Dwgs.User) (width 0.2))
